File: LED_Panel.sch (KiCad schematic (older format))
At the start: 0 parts

Commit message: Implemented the first version of the Panel-Driver
Parts:
- added C? (x2): 100nF, Capacitors_SMD:C_0805_HandSoldering, symbol C_Small
- added C?: 22nF, Capacitors_SMD:C_0805_HandSoldering, symbol C_Small
- added C?: 1μF, Capacitors_SMD:C_1206_HandSoldering, symbol C_Small
- added D?: D_Schot, Diodes_SMD:D_SOD-123, symbol D_Schottky
- added J?: Rotated_Barrel, symbol Rotated_Barrel
- added L?: 33μH, symbol L
- added R?: 162k, Resistors_SMD:R_0805_HandSoldering, symbol R
- added R?: 0R16, Resistors_SMD:R_0805_HandSoldering, symbol R
- added U?: LM3406HV, symbol LM3406HV
Connections:
- new net: R?.2, U?.10 (RON)
- new net: C?.1, U?.9 (COMP)
- new net: C?.1, U?.11 (VCC)
- new net: C?.2, D?.1 (K), L?.1, U?.1 (SW), U?.2 (SW)
- new net: C?.1, U?.3 (BOOT)
- new net: J?.1, L?.2, U?.5 (VOUT)
- new net: J?.2, J?.3, R?.1, U?.6 (CS)
- new net 48V: C?.1, R?.1, U?.12 (VINS), U?.13 (VIN), U?.14 (VIN)
- new net CONTROL: U?.8 (DIM)
- new net GND: C?.2, C?.2, C?.2, D?.2 (A), R?.2, U?.7 (GND)

Commit message: Added a missing datasheet
Parts:
- removed U?: LM3406HV, symbol LM3406HV
- added U?: LM3406HV, symbol LM3406HV
Connections:
- net 48V: now also U?.12 (VINS), U?.13 (VIN), U?.14 (VIN)
- net CONTROL: now also U?.8 (DIM)
- net GND: now also U?.7 (GND)
- net at R?.2: now also U?.10 (RON)
- net at C?.1: now also U?.9 (COMP)
- net at C?.1: now also U?.11 (VCC)
- net at C?.2, D?.1 (K), L?.1: now also U?.1 (SW), U?.2 (SW)
- net at C?.1: now also U?.3 (BOOT)
- net at J?.1, L?.2: now also U?.5 (VOUT)
- net at J?.2, J?.3, R?.1: now also U?.6 (CS)
Changed lines of the file:
@@
 $Descr A4 11693 8268
 encoding utf-8
-Sheet 4 5
+Sheet 3 5
 Title ""
 Date ""
@@
 AR Path="/5A4C3F5F/5A777BDD" Ref="#PWR043"  Part="1"
 AR Path="/5A4C34AF/5A777BDD" Ref="#PWR038"  Part="1"
-F 0 "#PWR043" H 1700 2450 50  0001 C CNN
+F 0 "#PWR038" H 1700 2450 50  0001 C CNN
 F 1 "GND" H 1700 2550 50  0000 C CNN
 F 2 "" H 1700 2700 50  0001 C CNN
@@
 AR Path="/5A4C3F5F/5A777CDA" Ref="#PWR044"  Part="1"
 AR Path="/5A4C34AF/5A777CDA" Ref="#PWR039"  Part="1"
-F 0 "#PWR044" H 2900 2450 50  0001 C CNN
+F 0 "#PWR039" H 2900 2450 50  0001 C CNN
 F 1 "GND" H 2900 2550 50  0000 C CNN
 F 2 "" H 2900 2700 50  0001 C CNN
 F 3 "" H 2900 2700 50  0001 C CNN
 	1    2900 2700
-	1    0    0    -1
-$EndComp
-$Comp
-L LM3406HV U?
-U 1 1 5A777F60
-P 2300 1900
-AR Path="/5A4C3F5F/5A777F60" Ref="U?"  Part="1"
-AR Path="/5A4C34AF/5A777F60" Ref="U?"  Part="1"
-F 0 "U?" H 2700 1350 60  0000 C CNN
-F 1 "LM3406HV" H 2100 2450 60  0000 C CNN
-F 2 "" H 2300 2500 60  0001 C CNN
-F 3 "" H 2300 2500 60  0001 C CNN
-	1    2300 1900
 	1    0    0    -1
 $EndComp
@@
 AR Path="/5A4C3F5F/5A777FA3" Ref="#PWR045"  Part="1"
 AR Path="/5A4C34AF/5A777FA3" Ref="#PWR040"  Part="1"
-F 0 "#PWR045" H 2300 2450 50  0001 C CNN
+F 0 "#PWR040" H 2300 2450 50  0001 C CNN
 F 1 "GND" H 2300 2550 50  0000 C CNN
 F 2 "" H 2300 2700 50  0001 C CNN
@@
 AR Path="/5A4C3F5F/5A778B62" Ref="#PWR046"  Part="1"
 AR Path="/5A4C34AF/5A778B62" Ref="#PWR041"  Part="1"
-F 0 "#PWR046" H 3200 2450 50  0001 C CNN
+F 0 "#PWR041" H 3200 2450 50  0001 C CNN
 F 1 "GND" H 3200 2550 50  0000 C CNN
 F 2 "" H 3200 2700 50  0001 C CNN
@@
 AR Path="/5A4C34AF/5A77A9CB" Ref="#PWR042"  Part="1"
 AR Path="/5A4C3F5F/5A77A9CB" Ref="#PWR047"  Part="1"
-F 0 "#PWR047" H 3650 2450 50  0001 C CNN
+F 0 "#PWR042" H 3650 2450 50  0001 C CNN
 F 1 "GND" H 3650 2550 50  0000 C CNN
 F 2 "" H 3650 2700 50  0001 C CNN
@@
 Wire Wire Line
 	1200 2100 1750 2100
+$Comp
+L LM3406HV U?
+U 1 1 5A77E620
+P 2300 1900
+F 0 "U?" H 2700 1350 60  0000 C CNN
+F 1 "LM3406HV" H 2100 2450 60  0000 C CNN
+F 2 "" H 2300 2500 60  0001 C CNN
+F 3 "http://www.ti.com/lit/ds/symlink/lm3406.pdf" H 2300 2500 60  0001 C CNN
+F 4 "https://www.digikey.com/product-detail/en/texas-instruments/LM3406HVMHX-NOPB/LM3406HVMHX-NOPBCT-ND/3526958" H 2300 1900 60  0001 C CNN "Digikey"
+	1    2300 1900
+	1    0    0    -1
+$EndComp
 $EndSCHEMATC

Commit message: Major changes, especially to the 12V-Rail
Other:
- note added: "Panel-Driver"
- moved on the sheet: C?, D?, J?, L?, R?, U?
