File: RGB.sch (KiCad schematic (older format))
At the start: 0 parts

Commit message: add preliminary RGB schematic
Parts:
- added D?: LED_ARGB, symbol LED_ARGB
- added Q? (x3): IRLB8721PBF, TO_SOT_Packages_THT:TO-220_Vertical, symbol IRLB8721PBF
Connections:
- new net: D?.2 (RK), Q?.2 (D)
- new net: D?.3 (GK), Q?.2 (D)
- new net: D?.4 (BK), Q?.2 (D)
- new net +12V: D?.1 (A)
- new net B_RGB: Q?.1 (G)
- new net GND: Q?.3 (S), Q?.3 (S), Q?.3 (S)
- new net G_RGB: Q?.1 (G)
- new net R_RGB: Q?.1 (G)
Other:
- note added: "TODO: Pinout von RGB LED Überprüfen"
Changed lines of the file:
@@
 Comment4 ""
 $EndDescr
+Text HLabel 4950 2500 0    60   Input ~ 0
+R_RGB
+Text HLabel 4950 3500 0    60   Input ~ 0
+G_RGB
+Text HLabel 4950 3000 0    60   Input ~ 0
+B_RGB
+$Comp
+L IRLB8721PBF Q?
+U 1 1 5A74E040
+P 5600 3450
+F 0 "Q?" H 5850 3525 50  0000 L CNN
+F 1 "IRLB8721PBF" H 5850 3450 50  0000 L CNN
+F 2 "TO_SOT_Packages_THT:TO-220_Vertical" H 5850 3375 50  0001 L CIN
+F 3 "" H 5600 3450 50  0001 L CNN
+	1    5600 3450
+	1    0    0    -1
+$EndComp
+$Comp
+L IRLB8721PBF Q?
+U 1 1 5A74E06E
+P 6000 2950
+F 0 "Q?" H 6250 3025 50  0000 L CNN
+F 1 "IRLB8721PBF" H 6250 2950 50  0000 L CNN
+F 2 "TO_SOT_Packages_THT:TO-220_Vertical" H 6250 2875 50  0001 L CIN
+F 3 "" H 6000 2950 50  0001 L CNN
+	1    6000 2950
+	1    0    0    -1
+$EndComp
+$Comp
+L IRLB8721PBF Q?
+U 1 1 5A74E0B0
+P 6400 2450
+F 0 "Q?" H 6650 2525 50  0000 L CNN
+F 1 "IRLB8721PBF" H 6650 2450 50  0000 L CNN
+F 2 "TO_SOT_Packages_THT:TO-220_Vertical" H 6650 2375 50  0001 L CIN
+F 3 "" H 6400 2450 50  0001 L CNN
+	1    6400 2450
+	1    0    0    -1
+$EndComp
+$Comp
+L LED_ARGB D?
+U 1 1 5A74E2BA
+P 6100 2050
+F 0 "D?" H 6100 2420 50  0000 C CNN
+F 1 "LED_ARGB" H 6100 1700 50  0000 C CNN
+F 2 "" H 6100 2000 50  0001 C CNN
+F 3 "" H 6100 2000 50  0001 C CNN
+	1    6100 2050
+	0    -1   -1   0
+$EndComp
+$Comp
+L +12V #PWR?
+U 1 1 5A74E6BA
+P 6100 1850
+F 0 "#PWR?" H 6100 1700 50  0001 C CNN
+F 1 "+12V" H 6100 1990 50  0000 C CNN
+F 2 "" H 6100 1850 50  0001 C CNN
+F 3 "" H 6100 1850 50  0001 C CNN
+	1    6100 1850
+	1    0    0    -1
+$EndComp
+Wire Wire Line
+	5700 2250 5900 2250
+Wire Wire Line
+	4950 2500 6200 2500
+Text Notes 6600 2000 0    60   ~ 0
+TODO: Pinout von RGB LED Überprüfen
+Wire Wire Line
+	4950 3000 5800 3000
+Wire Wire Line
+	4950 3500 5400 3500
+Wire Wire Line
+	6300 2250 6500 2250
+$Comp
+L GND #PWR?
+U 1 1 5A74EA81
+P 6500 2650
+F 0 "#PWR?" H 6500 2400 50  0001 C CNN
+F 1 "GND" H 6500 2500 50  0000 C CNN
+F 2 "" H 6500 2650 50  0001 C CNN
+F 3 "" H 6500 2650 50  0001 C CNN
+	1    6500 2650
+	1    0    0    -1
+$EndComp
+$Comp
+L GND #PWR?
+U 1 1 5A74EA9D
+P 6100 3150
+F 0 "#PWR?" H 6100 2900 50  0001 C CNN
+F 1 "GND" H 6100 3000 50  0000 C CNN
+F 2 "" H 6100 3150 50  0001 C CNN
+F 3 "" H 6100 3150 50  0001 C CNN
+	1    6100 3150
+	1    0    0    -1
+$EndComp
+$Comp
+L GND #PWR?
+U 1 1 5A74EAB9
+P 5700 3650
+F 0 "#PWR?" H 5700 3400 50  0001 C CNN
+F 1 "GND" H 5700 3500 50  0000 C CNN
+F 2 "" H 5700 3650 50  0001 C CNN
+F 3 "" H 5700 3650 50  0001 C CNN
+	1    5700 3650
+	1    0    0    -1
+$EndComp
+Wire Wire Line
+	5700 2250 5700 3250
+Wire Wire Line
+	6100 2250 6100 2750
 $EndSCHEMATC

Commit message: Major changes, especially to the 12V-Rail
Parts:
- removed Q? (x3): IRLB8721PBF, TO_SOT_Packages_THT:TO-220_Vertical, symbol IRLB8721PBF
- added Q? (x3): DMG2302UK, TO_SOT_Packages_SMD:SOT-23, symbol 2N7002
Connections:
- net B_RGB: now also Q?.1 (G)
- net GND: now also Q?.2 (S), Q?.2 (S), Q?.2 (S)
- net G_RGB: now also Q?.1 (G)
- net R_RGB: now also Q?.1 (G)
- net at D?.2 (RK): now also Q?.3 (D)
- net at D?.3 (GK): now also Q?.3 (D)
- net at D?.4 (BK): now also Q?.3 (D)
Other:
- note added: "RGB-Drivers"
- note removed: "TODO: Pinout von RGB LED Überprüfen"
- moved on the sheet: D?
Changed lines of the file:
@@
 LIBS:ledDriver
 LIBS:jacks
+LIBS:sensors
 LIBS:Hardware-cache
 EELAYER 25 0
@@
 Comment4 ""
 $EndDescr
-Text HLabel 4950 2500 0    60   Input ~ 0
+Text HLabel 950  1350 0    60   Input ~ 0
 R_RGB
-Text HLabel 4950 3500 0    60   Input ~ 0
+Text HLabel 850  2350 0    60   Input ~ 0
+B_RGB
+Text HLabel 900  1850 0    60   Input ~ 0
 G_RGB
-Text HLabel 4950 3000 0    60   Input ~ 0
-B_RGB
-$Comp
-L IRLB8721PBF Q?
-U 1 1 5A74E040
-P 5600 3450
-F 0 "Q?" H 5850 3525 50  0000 L CNN
-F 1 "IRLB8721PBF" H 5850 3450 50  0000 L CNN
-F 2 "TO_SOT_Packages_THT:TO-220_Vertical" H 5850 3375 50  0001 L CIN
-F 3 "" H 5600 3450 50  0001 L CNN
-	1    5600 3450
-	1    0    0    -1
-$EndComp
-$Comp
-L IRLB8721PBF Q?
-U 1 1 5A74E06E
-P 6000 2950
-F 0 "Q?" H 6250 3025 50  0000 L CNN
-F 1 "IRLB8721PBF" H 6250 2950 50  0000 L CNN
-F 2 "TO_SOT_Packages_THT:TO-220_Vertical" H 6250 2875 50  0001 L CIN
-F 3 "" H 6000 2950 50  0001 L CNN
-	1    6000 2950
-	1    0    0    -1
-$EndComp
-$Comp
-L IRLB8721PBF Q?
-U 1 1 5A74E0B0
-P 6400 2450
-F 0 "Q?" H 6650 2525 50  0000 L CNN
-F 1 "IRLB8721PBF" H 6650 2450 50  0000 L CNN
-F 2 "TO_SOT_Packages_THT:TO-220_Vertical" H 6650 2375 50  0001 L CIN
-F 3 "" H 6400 2450 50  0001 L CNN
-	1    6400 2450
-	1    0    0    -1
-$EndComp
 $Comp
 L LED_ARGB D?
 U 1 1 5A74E2BA
-P 6100 2050
-F 0 "D?" H 6100 2420 50  0000 C CNN
-F 1 "LED_ARGB" H 6100 1700 50  0000 C CNN
-F 2 "" H 6100 2000 50  0001 C CNN
-F 3 "" H 6100 2000 50  0001 C CNN
-	1    6100 2050
+P 2000 900
+F 0 "D?" H 2000 1270 50  0000 C CNN
+F 1 "LED_ARGB" H 2000 550 50  0000 C CNN
+F 2 "" H 2000 850 50  0001 C CNN
+F 3 "" H 2000 850 50  0001 C CNN
+	1    2000 900
 	0    -1   -1   0
 $EndComp
@@
 L +12V #PWR048
 U 1 1 5A74E6BA
-P 6100 1850
-F 0 "#PWR048" H 6100 1700 50  0001 C CNN
-F 1 "+12V" H 6100 1990 50  0000 C CNN
-F 2 "" H 6100 1850 50  0001 C CNN
-F 3 "" H 6100 1850 50  0001 C CNN
-	1    6100 1850
+P 2000 700
+F 0 "#PWR048" H 2000 550 50  0001 C CNN
+F 1 "+12V" H 2000 840 50  0000 C CNN
+F 2 "" H 2000 700 50  0001 C CNN
+F 3 "" H 2000 700 50  0001 C CNN
+	1    2000 700
 	1    0    0    -1
 $EndComp
 Wire Wire Line
-	5700 2250 5900 2250
+	1600 1100 1800 1100
 Wire Wire Line
-	4950 2500 6200 2500
-Text Notes 6600 2000 0    60   ~ 0
-TODO: Pinout von RGB LED Überprüfen
+	950  1350 2100 1350
 Wire Wire Line
-	4950 3000 5800 3000
+	900  1850 1700 1850
 Wire Wire Line
-	4950 3500 5400 3500
-Wire Wire Line
-	6300 2250 6500 2250
+	850  2350 1300 2350
 $Comp
 L GND #PWR049
 U 1 1 5A74EA81
-P 6500 2650
-F 0 "#PWR049" H 6500 2400 50  0001 C CNN
-F 1 "GND" H 6500 2500 50  0000 C CNN
-F 2 "" H 6500 2650 50  0001 C CNN
-F 3 "" H 6500 2650 50  0001 C CNN
-	1    6500 2650
+P 2400 1550
+F 0 "#PWR049" H 2400 1300 50  0001 C CNN
+F 1 "GND" H 2400 1400 50  0000 C CNN
+F 2 "" H 2400 1550 50  0001 C CNN
+F 3 "" H 2400 1550 50  0001 C CNN
+	1    2400 1550
 	1    0    0    -1
 $EndComp
@@
 L GND #PWR050
 U 1 1 5A74EA9D
-P 6100 3150
-F 0 "#PWR050" H 6100 2900 50  0001 C CNN
-F 1 "GND" H 6100 3000 50  0000 C CNN
-F 2 "" H 6100 3150 50  0001 C CNN
-F 3 "" H 6100 3150 50  0001 C CNN
-	1    6100 3150
+P 2000 2050
+F 0 "#PWR050" H 2000 1800 50  0001 C CNN
+F 1 "GND" H 2000 1900 50  0000 C CNN
+F 2 "" H 2000 2050 50  0001 C CNN
+F 3 "" H 2000 2050 50  0001 C CNN
+	1    2000 2050
 	1    0    0    -1
 $EndComp
@@
 L GND #PWR051
 U 1 1 5A74EAB9
-P 5700 3650
-F 0 "#PWR051" H 5700 3400 50  0001 C CNN
-F 1 "GND" H 5700 3500 50  0000 C CNN
-F 2 "" H 5700 3650 50  0001 C CNN
-F 3 "" H 5700 3650 50  0001 C CNN
-	1    5700 3650
+P 1600 2550
+F 0 "#PWR051" H 1600 2300 50  0001 C CNN
+F 1 "GND" H 1600 2400 50  0000 C CNN
+F 2 "" H 1600 2550 50  0001 C CNN
+F 3 "" H 1600 2550 50  0001 C CNN
+	1    1600 2550
 	1    0    0    -1
 $EndComp
 Wire Wire Line
-	5700 2250 5700 3250
+	1600 1100 1600 2150
 Wire Wire Line
-	6100 2250 6100 2750
+	2000 1100 2000 1650
+$Comp
+L 2N7002 Q?
+U 1 1 5A83A492
+P 1500 2350
+F 0 "Q?" H 1700 2425 50  0000 L CNN
+F 1 "DMG2302UK" H 1700 2350 50  0000 L CNN
+F 2 "TO_SOT_Packages_SMD:SOT-23" H 1700 2275 50  0001 L CIN
+F 3 "https://www.diodes.com/assets/Datasheets/DMG2302UK.pdf" H 1500 2350 50  0001 L CNN
+F 4 "https://www.digikey.com/product-detail/en/diodes-incorporated/DMG2302UK-7/DMG2302UK-7DICT-ND/6010163" H 1500 2350 60  0001 C CNN "Digikey"
+	1    1500 2350
+	1    0    0    -1
+$EndComp
+$Comp
+L 2N7002 Q?
+U 1 1 5A83A790
+P 1900 1850
+F 0 "Q?" H 2100 1925 50  0000 L CNN
+F 1 "DMG2302UK" H 2100 1850 50  0000 L CNN
+F 2 "TO_SOT_Packages_SMD:SOT-23" H 2100 1775 50  0001 L CIN
+F 3 "https://www.diodes.com/assets/Datasheets/DMG2302UK.pdf" H 1900 1850 50  0001 L CNN
+F 4 "https://www.digikey.com/product-detail/en/diodes-incorporated/DMG2302UK-7/DMG2302UK-7DICT-ND/6010163" H 1900 1850 60  0001 C CNN "Digikey"
+	1    1900 1850
+	1    0    0    -1
+$EndComp
+$Comp
+L 2N7002 Q?
+U 1 1 5A83A7DA
+P 2300 1350
+F 0 "Q?" H 2500 1425 50  0000 L CNN
+F 1 "DMG2302UK" H 2500 1350 50  0000 L CNN
+F 2 "TO_SOT_Packages_SMD:SOT-23" H 2500 1275 50  0001 L CIN
+F 3 "https://www.diodes.com/assets/Datasheets/DMG2302UK.pdf" H 2300 1350 50  0001 L CNN
+F 4 "https://www.digikey.com/product-detail/en/diodes-incorporated/DMG2302UK-7/DMG2302UK-7DICT-ND/6010163" H 2300 1350 60  0001 C CNN "Digikey"
+	1    2300 1350
+	1    0    0    -1
+$EndComp
+Wire Wire Line
+	2400 1150 2400 1100
+Wire Wire Line
+	2400 1100 2200 1100
+Text Notes 460  620  0    120  ~ 0
+RGB-Drivers
+Wire Notes Line
+	475  2750 3000 2750
+Wire Notes Line
+	3000 2750 3000 475
 $EndSCHEMATC
