File: RGB.sch (KiCad schematic (older format))
At the start: 7 parts, among them J8 LEDs, Q1 DMG2302UK, Q2 DMG2302UK, Q3 DMG2302UK

Commit message: Footprint-Association: 90%
Parts:
- J9: renamed from J8; footprint (none) -> Connectors_Terminal_Blocks:TerminalBlock_bornier-4_P5.08mm
Changed lines of the file:
@@
 G_RGB
 $Comp
-L +12V #PWR70
+L +12V #PWR075
 U 1 1 5A83A3DF
 P 2475 950
-F 0 "#PWR70" H 2475 800 50  0001 C CNN
+F 0 "#PWR075" H 2475 800 50  0001 C CNN
 F 1 "+12V" H 2475 1090 50  0000 C CNN
 F 2 "" H 2475 950 50  0001 C CNN
@@
 	1325 1900 1775 1900
 $Comp
-L GND #PWR71
+L GND #PWR076
 U 1 1 5A83A3E9
 P 2475 1600
-F 0 "#PWR71" H 2475 1350 50  0001 C CNN
+F 0 "#PWR076" H 2475 1350 50  0001 C CNN
 F 1 "GND" H 2475 1450 50  0000 C CNN
 F 2 "" H 2475 1600 50  0001 C CNN
@@
 $EndComp
 $Comp
-L GND #PWR72
+L GND #PWR077
 U 1 1 5A83A3EF
 P 2075 2100
-F 0 "#PWR72" H 2075 1850 50  0001 C CNN
+F 0 "#PWR077" H 2075 1850 50  0001 C CNN
 F 1 "GND" H 2075 1950 50  0000 C CNN
 F 2 "" H 2075 2100 50  0001 C CNN
@@
 $EndComp
 $Comp
-L GND #PWR73
+L GND #PWR078
 U 1 1 5A83A3F5
 P 1675 2600
-F 0 "#PWR73" H 1675 2350 50  0001 C CNN
+F 0 "#PWR078" H 1675 2350 50  0001 C CNN
 F 1 "GND" H 1675 2450 50  0000 C CNN
 F 2 "" H 1675 2600 50  0001 C CNN
@@
 	1025 2400 875  2400
 $Comp
-L Screw_Terminal_01x04 J8
+L Screw_Terminal_01x04 J9
 U 1 1 5A84BDDF
 P 2025 850
-F 0 "J8" H 2025 1050 50  0000 C CNN
+F 0 "J9" H 2025 1050 50  0000 C CNN
 F 1 "LEDs" H 2025 550 50  0000 C CNN
-F 2 "" H 2025 850 50  0001 C CNN
+F 2 "Connectors_Terminal_Blocks:TerminalBlock_bornier-4_P5.08mm" H 2025 850 50  0001 C CNN
 F 3 "" H 2025 850 50  0001 C CNN
 	1    2025 850

Commit message: Changed the 5V-Regulator
Parts:
- J9: symbol Screw_Terminal_01x04 -> Connector:Screw_Terminal_01x04
- Q1, Q2, Q3: symbol 2N7002 -> Transistor:2N7002
- R17, R18, R19: symbol R -> device:R
Changed lines of the file:
@@
-EESchema Schematic File Version 2
-LIBS:power
-LIBS:device
-LIBS:switches
-LIBS:transistors
-LIBS:conn
-LIBS:linear
-LIBS:regul
-LIBS:74xx
-LIBS:analog_switches
-LIBS:texas
-LIBS:interface
-LIBS:philips
-LIBS:cypress
-LIBS:siliconi
-LIBS:opto
-LIBS:contrib
-LIBS:stm32s
-LIBS:transceiver
-LIBS:switchingR
-LIBS:ledDriver
-LIBS:jacks
-LIBS:sensors
+EESchema Schematic File Version 4
 LIBS:Hardware-cache
-EELAYER 25 0
+EELAYER 26 0
 EELAYER END
 $Descr A4 11693 8268
@@
 G_RGB
 $Comp
-L +12V #PWR075
+L power:+12V #PWR075
 U 1 1 5A83A3DF
 P 2475 950
@@
 	1325 1900 1775 1900
 $Comp
-L GND #PWR076
+L power:GND #PWR076
 U 1 1 5A83A3E9
 P 2475 1600
@@
 $EndComp
 $Comp
-L GND #PWR077
+L power:GND #PWR077
 U 1 1 5A83A3EF
 P 2075 2100
@@
 $EndComp
 $Comp
-L GND #PWR078
+L power:GND #PWR078
 U 1 1 5A83A3F5
 P 1675 2600
@@
 	1675 1150 1675 2200
 $Comp
-L 2N7002 Q3
+L Transistor:2N7002 Q3
 U 1 1 5A83A3FE
 P 1575 2400
@@
 $EndComp
 $Comp
-L 2N7002 Q2
+L Transistor:2N7002 Q2
 U 1 1 5A83A406
 P 1975 1900
@@
 $EndComp
 $Comp
-L 2N7002 Q1
+L Transistor:2N7002 Q1
 U 1 1 5A83A40E
 P 2375 1400
@@
 	1325 2400 1375 2400
 $Comp
-L R R17
+L device:R R17
 U 1 1 5A8936F2
 P 1175 1400
@@
 	1325 1400 2175 1400
 $Comp
-L R R18
+L device:R R18
 U 1 1 5A8938B9
 P 1175 1900
@@
 	1025 1900 925  1900
 $Comp
-L R R19
+L device:R R19
 U 1 1 5A8939A3
 P 1175 2400
@@
 	1025 2400 875  2400
 $Comp
-L Screw_Terminal_01x04 J9
+L Connector:Screw_Terminal_01x04 J9
 U 1 1 5A84BDDF
 P 2025 850

Commit message: Updated to the new libraries
Parts:
- J9: symbol Connector:Screw_Terminal_01x04 -> Connector_Specialized:Screw_Terminal_01x04
- Q1: renamed from Q3; symbol Transistor:2N7002 -> Transistor_FET:2N7002
- Q2: symbol Transistor:2N7002 -> Transistor_FET:2N7002
- Q3: renamed from Q1; symbol Transistor:2N7002 -> Transistor_FET:2N7002
- R15: renamed from R17; symbol device:R -> Device:R
- R16: renamed from R18; symbol device:R -> Device:R
- R17: renamed from R19; symbol device:R -> Device:R
Changed lines of the file:
@@
 G_RGB
 $Comp
-L power:+12V #PWR075
+L power:+12V #PWR072
 U 1 1 5A83A3DF
 P 2475 950
-F 0 "#PWR075" H 2475 800 50  0001 C CNN
+F 0 "#PWR072" H 2475 800 50  0001 C CNN
 F 1 "+12V" H 2475 1090 50  0000 C CNN
 F 2 "" H 2475 950 50  0001 C CNN
@@
 	1325 1900 1775 1900
 $Comp
-L power:GND #PWR076
+L power:GND #PWR073
 U 1 1 5A83A3E9
 P 2475 1600
-F 0 "#PWR076" H 2475 1350 50  0001 C CNN
+F 0 "#PWR073" H 2475 1350 50  0001 C CNN
 F 1 "GND" H 2475 1450 50  0000 C CNN
 F 2 "" H 2475 1600 50  0001 C CNN
@@
 $EndComp
 $Comp
-L power:GND #PWR077
+L power:GND #PWR071
 U 1 1 5A83A3EF
 P 2075 2100
-F 0 "#PWR077" H 2075 1850 50  0001 C CNN
+F 0 "#PWR071" H 2075 1850 50  0001 C CNN
 F 1 "GND" H 2075 1950 50  0000 C CNN
 F 2 "" H 2075 2100 50  0001 C CNN
@@
 $EndComp
 $Comp
-L power:GND #PWR078
+L power:GND #PWR070
 U 1 1 5A83A3F5
 P 1675 2600
-F 0 "#PWR078" H 1675 2350 50  0001 C CNN
+F 0 "#PWR070" H 1675 2350 50  0001 C CNN
 F 1 "GND" H 1675 2450 50  0000 C CNN
 F 2 "" H 1675 2600 50  0001 C CNN
@@
 	1675 1150 1675 2200
 $Comp
-L Transistor:2N7002 Q3
+L Transistor_FET:2N7002 Q1
 U 1 1 5A83A3FE
 P 1575 2400
-F 0 "Q3" H 1775 2475 50  0000 L CNN
+F 0 "Q1" H 1775 2475 50  0000 L CNN
 F 1 "DMG2302UK" H 1775 2400 50  0000 L CNN
 F 2 "TO_SOT_Packages_SMD:SOT-23" H 1775 2325 50  0001 L CIN
@@
 $EndComp
 $Comp
-L Transistor:2N7002 Q2
+L Transistor_FET:2N7002 Q2
 U 1 1 5A83A406
 P 1975 1900
@@
 $EndComp
 $Comp
-L Transistor:2N7002 Q1
+L Transistor_FET:2N7002 Q3
 U 1 1 5A83A40E
 P 2375 1400
-F 0 "Q1" H 2575 1475 50  0000 L CNN
+F 0 "Q3" H 2575 1475 50  0000 L CNN
 F 1 "DMG2302UK" H 2575 1400 50  0000 L CNN
 F 2 "TO_SOT_Packages_SMD:SOT-23" H 2575 1325 50  0001 L CIN
@@
 	1325 2400 1375 2400
 $Comp
-L device:R R17
+L Device:R R15
 U 1 1 5A8936F2
 P 1175 1400
-F 0 "R17" V 1255 1400 50  0000 C CNN
+F 0 "R15" V 1255 1400 50  0000 C CNN
 F 1 "165" V 1175 1400 50  0000 C CNN
 F 2 "Resistors_SMD:R_0603" V 1105 1400 50  0001 C CNN
@@
 	1325 1400 2175 1400
 $Comp
-L device:R R18
+L Device:R R16
 U 1 1 5A8938B9
 P 1175 1900
-F 0 "R18" V 1255 1900 50  0000 C CNN
+F 0 "R16" V 1255 1900 50  0000 C CNN
 F 1 "165" V 1175 1900 50  0000 C CNN
 F 2 "Resistors_SMD:R_0603" V 1105 1900 50  0001 C CNN
@@
 	1025 1900 925  1900
 $Comp
-L device:R R19
+L Device:R R17
 U 1 1 5A8939A3
 P 1175 2400
-F 0 "R19" V 1255 2400 50  0000 C CNN
+F 0 "R17" V 1255 2400 50  0000 C CNN
 F 1 "165" V 1175 2400 50  0000 C CNN
 F 2 "Resistors_SMD:R_0603" V 1105 2400 50  0001 C CNN
@@
 	1025 2400 875  2400
 $Comp
-L Connector:Screw_Terminal_01x04 J9
+L Connector_Specialized:Screw_Terminal_01x04 J9
 U 1 1 5A84BDDF
 P 2025 850

Commit message: Changed the RJ45 to a Quad-Type
Parts:
- renumbered J9 to J8
Changed lines of the file:
@@
 G_RGB
 $Comp
-L power:+12V #PWR072
+L power:+12V #PWR075
 U 1 1 5A83A3DF
 P 2475 950
-F 0 "#PWR072" H 2475 800 50  0001 C CNN
+F 0 "#PWR075" H 2475 800 50  0001 C CNN
 F 1 "+12V" H 2475 1090 50  0000 C CNN
 F 2 "" H 2475 950 50  0001 C CNN
@@
 	1325 1900 1775 1900
 $Comp
-L power:GND #PWR073
+L power:GND #PWR076
 U 1 1 5A83A3E9
 P 2475 1600
-F 0 "#PWR073" H 2475 1350 50  0001 C CNN
+F 0 "#PWR076" H 2475 1350 50  0001 C CNN
 F 1 "GND" H 2475 1450 50  0000 C CNN
 F 2 "" H 2475 1600 50  0001 C CNN
@@
 $EndComp
 $Comp
-L power:GND #PWR071
+L power:GND #PWR074
 U 1 1 5A83A3EF
 P 2075 2100
-F 0 "#PWR071" H 2075 1850 50  0001 C CNN
+F 0 "#PWR074" H 2075 1850 50  0001 C CNN
 F 1 "GND" H 2075 1950 50  0000 C CNN
 F 2 "" H 2075 2100 50  0001 C CNN
@@
 $EndComp
 $Comp
-L power:GND #PWR070
+L power:GND #PWR073
 U 1 1 5A83A3F5
 P 1675 2600
-F 0 "#PWR070" H 1675 2350 50  0001 C CNN
+F 0 "#PWR073" H 1675 2350 50  0001 C CNN
 F 1 "GND" H 1675 2450 50  0000 C CNN
 F 2 "" H 1675 2600 50  0001 C CNN
@@
 	1025 2400 875  2400
 $Comp
-L Connector_Specialized:Screw_Terminal_01x04 J9
+L Connector_Specialized:Screw_Terminal_01x04 J8
 U 1 1 5A84BDDF
 P 2025 850
-F 0 "J9" H 2025 1050 50  0000 C CNN
+F 0 "J8" H 2025 1050 50  0000 C CNN
 F 1 "LEDs" H 2025 550 50  0000 C CNN
 F 2 "Connectors_Terminal_Blocks:TerminalBlock_bornier-4_P5.08mm" H 2025 850 50  0001 C CNN

Commit message: Made the Digikey more generic
Parts:
- Q1, Q2, Q3: Buy (none) -> https://www.digikey.com/product-detail/en/diodes-incorporat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; Digikey https://www.digikey.com/product-detail/en/diodes-incorporat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 -> (none)
Changed lines of the file:
@@
 F 2 "TO_SOT_Packages_SMD:SOT-23" H 1775 2325 50  0001 L CIN
 F 3 "https://www.diodes.com/assets/Datasheets/DMG2302UK.pdf" H 1575 2400 50  0001 L CNN
-F 4 "https://www.digikey.com/product-detail/en/diodes-incorporated/DMG2302UK-7/DMG2302UK-7DICT-ND/6010163" H 1575 2400 60  0001 C CNN "Digikey"
+F 4 "https://www.digikey.com/product-detail/en/diodes-incorporated/DMG2302UK-7/DMG2302UK-7DICT-ND/6010163" H 1575 2400 60  0001 C CNN "Buy"
 	1    1575 2400
 	1    0    0    -1
@@
 F 2 "TO_SOT_Packages_SMD:SOT-23" H 2175 1825 50  0001 L CIN
 F 3 "https://www.diodes.com/assets/Datasheets/DMG2302UK.pdf" H 1975 1900 50  0001 L CNN
-F 4 "https://www.digikey.com/product-detail/en/diodes-incorporated/DMG2302UK-7/DMG2302UK-7DICT-ND/6010163" H 1975 1900 60  0001 C CNN "Digikey"
+F 4 "https://www.digikey.com/product-detail/en/diodes-incorporated/DMG2302UK-7/DMG2302UK-7DICT-ND/6010163" H 1975 1900 60  0001 C CNN "Buy"
 	1    1975 1900
 	1    0    0    -1
@@
 F 2 "TO_SOT_Packages_SMD:SOT-23" H 2575 1325 50  0001 L CIN
 F 3 "https://www.diodes.com/assets/Datasheets/DMG2302UK.pdf" H 2375 1400 50  0001 L CNN
-F 4 "https://www.digikey.com/product-detail/en/diodes-incorporated/DMG2302UK-7/DMG2302UK-7DICT-ND/6010163" H 2375 1400 60  0001 C CNN "Digikey"
+F 4 "https://www.digikey.com/product-detail/en/diodes-incorporated/DMG2302UK-7/DMG2302UK-7DICT-ND/6010163" H 2375 1400 60  0001 C CNN "Buy"
 	1    2375 1400
 	1    0    0    -1

Commit message: Added Component-Associations (about 10% remaining)
Parts:
- R15, R16, R17: Buy (none) -> https://www.digikey.com/product-detail/en/yageo/RC0603FR-07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
Changed lines of the file:
@@
 F 2 "Resistors_SMD:R_0603" V 1105 1400 50  0001 C CNN
 F 3 "" H 1175 1400 50  0001 C CNN
+F 4 "https://www.digikey.com/product-detail/en/yageo/RC0603FR-07165RL/311-165HRCT-ND/729923" V 1175 1400 50  0001 C CNN "Buy"
 	1    1175 1400
 	0    1    1    0
@@
 F 2 "Resistors_SMD:R_0603" V 1105 1900 50  0001 C CNN
 F 3 "" H 1175 1900 50  0001 C CNN
+F 4 "https://www.digikey.com/product-detail/en/yageo/RC0603FR-07165RL/311-165HRCT-ND/729923" V 1175 1900 50  0001 C CNN "Buy"
 	1    1175 1900
 	0    1    1    0
@@
 F 2 "Resistors_SMD:R_0603" V 1105 2400 50  0001 C CNN
 F 3 "" H 1175 2400 50  0001 C CNN
+F 4 "https://www.digikey.com/product-detail/en/yageo/RC0603FR-07165RL/311-165HRCT-ND/729923" V 1175 2400 50  0001 C CNN "Buy"
 	1    1175 2400
 	0    1    1    0

Commit message: Added about 8% of the remaining components
Parts:
- renumbered J8 to J9, R15 to R19, R16 to R20, R17 to R21
Changed lines of the file:
@@
 G_RGB
 $Comp
-L power:+12V #PWR075
+L power:+12V #PWR078
 U 1 1 5A83A3DF
 P 2475 950
-F 0 "#PWR075" H 2475 800 50  0001 C CNN
+F 0 "#PWR078" H 2475 800 50  0001 C CNN
 F 1 "+12V" H 2475 1090 50  0000 C CNN
 F 2 "" H 2475 950 50  0001 C CNN
@@
 	1325 1900 1775 1900
 $Comp
-L power:GND #PWR076
+L power:GND #PWR079
 U 1 1 5A83A3E9
 P 2475 1600
-F 0 "#PWR076" H 2475 1350 50  0001 C CNN
+F 0 "#PWR079" H 2475 1350 50  0001 C CNN
 F 1 "GND" H 2475 1450 50  0000 C CNN
 F 2 "" H 2475 1600 50  0001 C CNN
@@
 $EndComp
 $Comp
-L power:GND #PWR074
+L power:GND #PWR077
 U 1 1 5A83A3EF
 P 2075 2100
-F 0 "#PWR074" H 2075 1850 50  0001 C CNN
+F 0 "#PWR077" H 2075 1850 50  0001 C CNN
 F 1 "GND" H 2075 1950 50  0000 C CNN
 F 2 "" H 2075 2100 50  0001 C CNN
@@
 $EndComp
 $Comp
-L power:GND #PWR073
+L power:GND #PWR076
 U 1 1 5A83A3F5
 P 1675 2600
-F 0 "#PWR073" H 1675 2350 50  0001 C CNN
+F 0 "#PWR076" H 1675 2350 50  0001 C CNN
 F 1 "GND" H 1675 2450 50  0000 C CNN
 F 2 "" H 1675 2600 50  0001 C CNN
@@
 	1325 2400 1375 2400
 $Comp
-L Device:R R15
+L Device:R R19
 U 1 1 5A8936F2
 P 1175 1400
-F 0 "R15" V 1255 1400 50  0000 C CNN
+F 0 "R19" V 1255 1400 50  0000 C CNN
 F 1 "165" V 1175 1400 50  0000 C CNN
 F 2 "Resistors_SMD:R_0603" V 1105 1400 50  0001 C CNN
@@
 	1325 1400 2175 1400
 $Comp
-L Device:R R16
+L Device:R R20
 U 1 1 5A8938B9
 P 1175 1900
-F 0 "R16" V 1255 1900 50  0000 C CNN
+F 0 "R20" V 1255 1900 50  0000 C CNN
 F 1 "165" V 1175 1900 50  0000 C CNN
 F 2 "Resistors_SMD:R_0603" V 1105 1900 50  0001 C CNN
@@
 	1025 1900 925  1900
 $Comp
-L Device:R R17
+L Device:R R21
 U 1 1 5A8939A3
 P 1175 2400
-F 0 "R17" V 1255 2400 50  0000 C CNN
+F 0 "R21" V 1255 2400 50  0000 C CNN
 F 1 "165" V 1175 2400 50  0000 C CNN
 F 2 "Resistors_SMD:R_0603" V 1105 2400 50  0001 C CNN
@@
 	1025 2400 875  2400
 $Comp
-L Connector_Specialized:Screw_Terminal_01x04 J8
+L Connector_Specialized:Screw_Terminal_01x04 J9
 U 1 1 5A84BDDF
 P 2025 850
-F 0 "J8" H 2025 1050 50  0000 C CNN
+F 0 "J9" H 2025 1050 50  0000 C CNN
 F 1 "LEDs" H 2025 550 50  0000 C CNN
 F 2 "Connectors_Terminal_Blocks:TerminalBlock_bornier-4_P5.08mm" H 2025 850 50  0001 C CNN

Commit message: Added Gate Pull-Downs
Parts:
- added R? (x3): 10k, Resistors_SMD:R_0603, symbol Device:R
Connections:
- wire segments 17 -> 23
Other:
- moved on the sheet: Q1, Q2, Q3
