File: Hardware.sch (KiCad schematic (older format))
At the start: 16 parts

Commit message: Unmerged the LED-Parts
Parts:
- C1, C2, C3, C4, C5: renamed from C?; footprint (none) -> Capacitors_SMD:C_0603
- R1, R2: renamed from R?; footprint (none) -> Resistors_SMD:R_0603
- U2: renamed from U?; footprint UFQFPN28 -> (none)
- gave numbers to parts that had none: 8
Connections:
- wire segments 153 -> 155

Commit message: Footprint-Association: 90%
Parts:
- removed J1: Screw_01x04, symbol Screw_Terminal_01x04
- added J5, J6: RJ45, RJ45:RJ45_9, symbol RJ45
- J1: renamed from J2; footprint (none) -> Socket_Strips:Socket_Strip_Straight_2x05_Pitch2.54mm
- J2: renamed from J3; footprint (none) -> Socket_Strips:Socket_Strip_Straight_1x05_Pitch2.54mm
- J3: renamed from J4; footprint (none) -> Socket_Strips:Socket_Strip_Straight_1x07_Pitch2.54mm
- J4: renamed from J5; footprint (none) -> Socket_Strips:Socket_Strip_Straight_2x04_Pitch2.54mm
- Y1: footprint (none) -> Crystals:Crystal_SMD_HC49-SD
Connections:
- net labels added: CAN_H, CAN_L, DMX_A, DMX_B
- wire segments 155 -> 167
- no-connect marks 1 -> 9

Commit message: Changed the 5V-Regulator
Parts:
- removed U1, U3: MCP9700AT-E/TT, TO_SOT_Packages_SMD:SOT-23, symbol MCP9700AT-E/TT
- added U1, U3: MCP9700T, TO_SOT_Packages_SMD:SOT-23, symbol mcp9700t:MCP9700T
- C1: symbol CP_Small -> device:CP_Small
- C2, C3, C4, C5: symbol C_Small -> device:C_Small
- J1: symbol Conn_02x05_Odd_Even -> Connector:Conn_02x05_Odd_Even
- J2: symbol Conn_01x05_Female -> Connector:Conn_01x05_Female
- J3: symbol Conn_01x07_Female -> Connector:Conn_01x07_Female
- J4: symbol Conn_02x04_Odd_Even -> Connector:Conn_02x05_Odd_Even
- J5, J6: symbol RJ45 -> Connector:RJ45
- R1: symbol R -> device:R
- R2: symbol R_Small -> device:R_Small
- U2: footprint (none) -> QFP:UFQFPN-28_4x4mm_Pitch0.5mm; symbol STM32F042G6Ux -> stm32s:STM32F042G6Ux
- Y1: symbol Crystal_Small -> device:Crystal_Small
Connections:
- wire segments 167 -> 190

Commit message: Minor Bugfixes
Parts:
- removed J4: ESP_Conn, Socket_Strips:Socket_Strip_Straight_2x04_Pitch2.54mm, symbol Connector:Conn_02x05_Odd_Even
- added J?: Conn_02x04, symbol Connector:Conn_02x04_Odd_Even
Changed lines of the file:
@@
 SWD_CLK
 NoConn ~ 4100 4150
-$Comp
-L Connector:Conn_02x05_Odd_Even J4
-U 1 1 5A8769E8
-P 4300 5650
-F 0 "J4" H 4350 5850 50  0000 C CNN
-F 1 "ESP_Conn" H 4350 5350 50  0000 C CNN
-F 2 "Socket_Strips:Socket_Strip_Straight_2x04_Pitch2.54mm" H 4300 5650 50  0001 C CNN
-F 3 "" H 4300 5650 50  0001 C CNN
-	1    4300 5650
-	1    0    0    -1
-$EndComp
 Text GLabel 4050 5550 0    60   Input ~ 0
 UART1_TX
@@
 U 1 1 5A85CDF5
 P 4050 6750
-F 0 "J5" H 4250 7250 50  0000 C CNN
-F 1 "RJ45" H 3900 7250 50  0000 C CNN
+F 0 "J5" H 4400 7250 50  0000 C CNN
+F 1 "RJ45" H 3750 7250 50  0000 C CNN
 F 2 "RJ45:RJ45_9" H 4050 6750 50  0001 C CNN
 F 3 "" H 4050 6750 50  0001 C CNN
@@
 U 1 1 5A85D43C
 P 5700 6750
-F 0 "J6" H 5900 7250 50  0000 C CNN
-F 1 "RJ45" H 5550 7250 50  0000 C CNN
+F 0 "J6" H 6050 7250 50  0000 C CNN
+F 1 "RJ45" H 5400 7250 50  0000 C CNN
 F 2 "RJ45:RJ45_9" H 5700 6750 50  0001 C CNN
 F 3 "" H 5700 6750 50  0001 C CNN
@@
 	1    0    0    -1
 $EndComp
+$Comp
+L Connector:Conn_02x04_Odd_Even J?
+U 1 1 5AA7F61D
+P 4300 5650
+F 0 "J?" H 4350 5967 50  0000 C CNN
+F 1 "Conn_02x04" H 4350 5876 50  0000 C CNN
+F 2 "" H 4300 5650 50  0001 C CNN
+F 3 "~" H 4300 5650 50  0001 C CNN
+	1    4300 5650
+	1    0    0    -1
+$EndComp

Commit message: Updated to the new libraries
Parts:
- C1: renamed from C4; symbol device:C_Small -> Device:C_Small
- C2: renamed from C3; symbol device:C_Small -> Device:C_Small
- C3: renamed from C5; symbol device:C_Small -> Device:C_Small
- C4: renamed from C1; symbol device:CP_Small -> Device:CP_Small
- C5: renamed from C2; symbol device:C_Small -> Device:C_Small
- J1: renamed from J5; symbol Connector:RJ45 -> Connector_Specialized:RJ45
- J2: renamed from J1; symbol Connector:Conn_02x05_Odd_Even -> Connector_Generic:Conn_02x05_Odd_Even
- J3: renamed from J?; symbol Connector:Conn_02x04_Odd_Even -> Connector_Generic:Conn_02x04_Odd_Even
- J4: renamed from J6; symbol Connector:RJ45 -> Connector_Specialized:RJ45
- J5: renamed from J2; symbol Connector:Conn_01x05_Female -> Connector_Specialized:Conn_01x05_Female
- J6: renamed from J3; symbol Connector:Conn_01x07_Female -> Connector_Specialized:Conn_01x07_Female
- R1: symbol device:R -> Device:R
- R2: symbol device:R_Small -> Device:R_Small
- U2: renamed from U1; value MCP9700T -> MCP9700T-ETT; symbol mcp9700t:MCP9700T -> Sensor_Temperature:MCP9700T-ETT
- U3: value MCP9700T -> MCP9700T-ETT; symbol mcp9700t:MCP9700T -> Sensor_Temperature:MCP9700T-ETT
- Y1: symbol device:Crystal_Small -> Device:Crystal_Small
- renumbered U2 to U1

Commit message: Added two additional RJ45-Ports
Parts:
- removed J1, J4: RJ45, RJ45:RJ45_9, symbol Connector_Specialized:RJ45
- added J? (x4): RJ45, RJ45:RJ45_9, symbol Connector_Specialized:RJ45
- added T? (x4): Test_Point, symbol Connector_Specialized:Test_Point
- C2: Digikey (none) -> https://www.digikey.com/product-detail/en/samsung-electro-m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
Connections:
- net labels added: RJ45-1, RJ45-2, RJ45-3, RJ45-4, RJ45-5, RJ45-6, RJ45-7, RJ45-8
- wire segments 190 -> 207
- no-connect marks 9 -> 1

Commit message: Changed the RJ45 to a Quad-Type
Parts:
- removed J? (x4): RJ45, RJ45:RJ45_9, symbol Connector_Specialized:RJ45
- added J1: RJ45-Quad, symbol connectors:RJ45-Quad
- gave numbers to parts that had none: 4
- renumbered J6 to J4

Commit message: Made the Digikey more generic
Parts:
- C2, C3: Buy (none) -> https://www.digikey.com/product-detail/en/samsung-electro-m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; Digikey https://www.digikey.com/product-detail/en/samsung-electro-m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 -> (none)
- U1: Buy (none) -> https://www.digikey.com/product-detail/en/stmicroelectronic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; Digikey https://www.digikey.com/product-detail/en/stmicroelectronic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 -> (none)
- U2, U3: Buy (none) -> https://www.digikey.com/product-detail/en/microchip-technol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; Digikey https://www.digikey.com/product-detail/en/microchip-technol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 -> (none)
- Y1: Buy (none) -> https://www.digikey.com/product-detail/en/abracon-llc/ABLS-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; Digikey https://www.digikey.com/product-detail/en/abracon-llc/ABLS-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 -> (none)
Changed lines of the file:
@@
 F 2 "QFP:UFQFPN-28_4x4mm_Pitch0.5mm" H 5850 3250 50  0001 R TNN
 F 3 "" H 4200 2350 50  0001 C CNN
-F 4 "https://www.digikey.com/product-detail/en/stmicroelectronics/STM32F042G6U6/497-17345-ND/5268192" H 4200 2350 60  0001 C CNN "Digikey"
+F 4 "https://www.digikey.com/product-detail/en/stmicroelectronics/STM32F042G6U6/497-17345-ND/5268192" H 4200 2350 60  0001 C CNN "Buy"
 	1    4200 2350
 	1    0    0    -1
@@
 F 2 "Crystals:Crystal_SMD_HC49-SD" H 1650 2000 50  0001 C CNN
 F 3 "" H 1650 2000 50  0001 C CNN
-F 4 "https://www.digikey.com/product-detail/en/abracon-llc/ABLS-8.000MHZ-B4-T/535-10212-1-ND/2184247" H 1650 2000 60  0001 C CNN "Digikey"
+F 4 "https://www.digikey.com/product-detail/en/abracon-llc/ABLS-8.000MHZ-B4-T/535-10212-1-ND/2184247" H 1650 2000 60  0001 C CNN "Buy"
 	1    1650 2000
 	0    1    1    0
@@
 F 2 "Capacitors_SMD:C_0603" H 1400 1850 50  0001 C CNN
 F 3 "" H 1400 1850 50  0001 C CNN
-F 4 "https://www.digikey.com/product-detail/en/samsung-electro-mechanics/CL21C150JBANNNC/1276-1163-1-ND/3889249" H 1400 1850 50  0001 C CNN "Digikey"
+F 4 "https://www.digikey.com/product-detail/en/samsung-electro-mechanics/CL21C150JBANNNC/1276-1163-1-ND/3889249" H 1400 1850 50  0001 C CNN "Buy"
 	1    1400 1850
 	0    1    1    0
@@
 F 2 "Capacitors_SMD:C_0603" H 1400 2150 50  0001 C CNN
 F 3 "" H 1400 2150 50  0001 C CNN
-F 4 "https://www.digikey.com/product-detail/en/samsung-electro-mechanics/CL21C150JBANNNC/1276-1163-1-ND/3889249" H 1400 2150 60  0001 C CNN "Digikey"
+F 4 "https://www.digikey.com/product-detail/en/samsung-electro-mechanics/CL21C150JBANNNC/1276-1163-1-ND/3889249" H 1400 2150 60  0001 C CNN "Buy"
 	1    1400 2150
 	0    1    1    0
@@
 F 2 "TO_SOT_Packages_SMD:SOT-23" H 7700 2300 50  0001 C CNN
 F 3 "" H 7550 2950 50  0001 C CNN
-F 4 "https://www.digikey.com/product-detail/en/microchip-technology/MCP9700T-E-TT/MCP9700T-E-TTCT-ND/1212545" H 7700 2700 50  0001 C CNN "Digikey"
+F 4 "https://www.digikey.com/product-detail/en/microchip-technology/MCP9700T-E-TT/MCP9700T-E-TTCT-ND/1212545" H 7700 2700 50  0001 C CNN "Buy"
 	1    7700 2700
 	1    0    0    -1
@@
 F 2 "TO_SOT_Packages_SMD:SOT-23" H 7700 950 50  0001 C CNN
 F 3 "" H 7550 1600 50  0001 C CNN
-F 4 "https://www.digikey.com/product-detail/en/microchip-technology/MCP9700T-E-TT/MCP9700T-E-TTCT-ND/1212545" H 7700 1350 50  0001 C CNN "Digikey"
+F 4 "https://www.digikey.com/product-detail/en/microchip-technology/MCP9700T-E-TT/MCP9700T-E-TTCT-ND/1212545" H 7700 1350 50  0001 C CNN "Buy"
 	1    7700 1350
 	1    0    0    -1
