File: Hardware.sch (KiCad schematic (older format))
At the start: 26 parts, among them J1 Power, J10 Conn_Extra_RJ45, J3 SWD_Conn, J4 Conn_02x04, J5 Spare_Conn, J6 Power_Conn, U1 STM32F042G6Ux, U2 MCP9700T-ETT, U3 MCP9700T-ETT, Y1 8MHz

Commit message: Realigned RJ45-Connector
Other:
- note removed: "specs auf shield überprüfen"
- moved on the sheet: J?A, J?B

Commit message: Added an additional capacitor next to the RGB-Strip
Parts:
- added C?: 4.7μF, Capacitor_SMD:C_0603_1608Metric, symbol Device:CP_Small
Connections:
- wire segments 224 -> 228
Other:
- moved on the sheet: C6, U2, U3

Commit message: Replaced the 10k-Resistor with one that is in stock
Parts:
- R1, R2, R?: Buy https://www.digikey.com/product-detail/en/yageo/RC0603FR-07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 -> https://www.digikey.com/product-detail/en/bourns-inc/CR0603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
Changed lines of the file:
@@
 F 2 "Resistor_SMD:R_0603_1608Metric" V 2280 3150 50  0001 C CNN
 F 3 "" H 2350 3150 50  0001 C CNN
-F 4 "https://www.digikey.com/product-detail/en/yageo/RC0603FR-0710KL/311-10.0KHRCT-ND/729827" V 2350 3150 50  0001 C CNN "Buy"
+F 4 "https://www.digikey.com/product-detail/en/bourns-inc/CR0603-FX-1002HLF/CR0603-FX-1002HLFCT-ND/3925297" V 2350 3150 50  0001 C CNN "Buy"
 	1    2350 3150
 	1    0    0    -1
@@
 F 2 "Resistor_SMD:R_0603_1608Metric" H 3475 4850 50  0001 C CNN
 F 3 "" H 3475 4850 50  0001 C CNN
-F 4 "https://www.digikey.com/product-detail/en/yageo/RC0603FR-0710KL/311-10.0KHRCT-ND/729827" H 3475 4850 50  0001 C CNN "Buy"
+F 4 "https://www.digikey.com/product-detail/en/bourns-inc/CR0603-FX-1002HLF/CR0603-FX-1002HLFCT-ND/3925297" H 3475 4850 50  0001 C CNN "Buy"
 	1    3475 4850
 	0    -1   -1   0
@@
 F 2 "Resistor_SMD:R_0603_1608Metric" V 780 1550 50  0001 C CNN
 F 3 "" H 850 1550 50  0001 C CNN
-F 4 "https://www.digikey.com/product-detail/en/yageo/RC0603FR-0710KL/311-10.0KHRCT-ND/729827" V 850 1550 50  0001 C CNN "Buy"
+F 4 "https://www.digikey.com/product-detail/en/bourns-inc/CR0603-FX-1002HLF/CR0603-FX-1002HLFCT-ND/3925297" V 850 1550 50  0001 C CNN "Buy"
 	1    850  1550
 	1    0    0    -1

Commit message: Replaced the 100nF Low-Voltage-Caps with one, which is still in stock
Parts:
- C1, C35, C5, C6: Buy https://www.digikey.com/product-detail/en/kemet/C0603C104K3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 -> https://www.digikey.com/product-detail/en/murata-electronic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
Changed lines of the file:
@@
 F 2 "Capacitor_SMD:C_0603_1608Metric" H 850 1900 50  0001 C CNN
 F 3 "" H 850 1900 50  0001 C CNN
-F 4 "https://www.digikey.com/product-detail/en/kemet/C0603C104K3RACTU/399-1281-1-ND/416057" H 850 1900 50  0001 C CNN "Buy"
+F 4 "https://www.digikey.com/product-detail/en/murata-electronics-north-america/GCM188R71C104KA37D/490-4774-1-ND/1641693" H 850 1900 50  0001 C CNN "Buy"
 	1    850  1900
 	1    0    0    -1
@@
 F 2 "Capacitor_SMD:C_0603_1608Metric" H 4000 1050 50  0001 C CNN
 F 3 "" H 4000 1050 50  0001 C CNN
-F 4 "https://www.digikey.com/product-detail/en/kemet/C0603C104K3RACTU/399-1281-1-ND/416057" V 4000 1050 50  0001 C CNN "Buy"
+F 4 "https://www.digikey.com/product-detail/en/murata-electronics-north-america/GCM188R71C104KA37D/490-4774-1-ND/1641693" V 4000 1050 50  0001 C CNN "Buy"
 	1    4000 1050
 	0    1    1    0
@@
 F 2 "" H 7075 5900 50  0001 C CNN
 F 3 "~" H 7075 5900 50  0001 C CNN
-F 4 "https://www.digikey.com/product-detail/en/kemet/C0603C104K3RACTU/399-1281-1-ND/416057" H 7075 5900 50  0001 C CNN "Buy"
+F 4 "https://www.digikey.com/product-detail/en/murata-electronics-north-america/GCM188R71C104KA37D/490-4774-1-ND/1641693" H 7075 5900 50  0001 C CNN "Buy"
 	1    7075 5900
 	1    0    0    -1
@@
 F 2 "Capacitor_SMD:C_0603_1608Metric" H 4700 1050 50  0001 C CNN
 F 3 "" H 4700 1050 50  0001 C CNN
-F 4 "https://www.digikey.com/product-detail/en/kemet/C0603C104K3RACTU/399-1281-1-ND/416057" V 4700 1050 50  0001 C CNN "Buy"
+F 4 "https://www.digikey.com/product-detail/en/murata-electronics-north-america/GCM188R71C104KA37D/490-4774-1-ND/1641693" V 4700 1050 50  0001 C CNN "Buy"
 	1    4700 1050
 	0    1    1    0

Commit message: Replaced the 15pF Low-Voltage-Caps with one, which is still in stock
Parts:
- C2, C3: Buy https://www.digikey.com/product-detail/en/samsung-electro-m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 -> https://www.digikey.com/product-detail/en/yageo/CC0603JRNPO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
Changed lines of the file:
@@
 F 2 "Capacitor_SMD:C_0603_1608Metric" H 1400 1850 50  0001 C CNN
 F 3 "" H 1400 1850 50  0001 C CNN
-F 4 "https://www.digikey.com/product-detail/en/samsung-electro-mechanics/CL10C150JB8NCNC/1276-2190-1-ND/3890276" H 1400 1850 50  0001 C CNN "Buy"
+F 4 "https://www.digikey.com/product-detail/en/yageo/CC0603JRNPO9BN150/311-1060-1-ND/302970" H 1400 1850 50  0001 C CNN "Buy"
 	1    1400 1850
 	0    1    1    0
@@
 F 2 "Capacitor_SMD:C_0603_1608Metric" H 1400 2150 50  0001 C CNN
 F 3 "" H 1400 2150 50  0001 C CNN
-F 4 "https://www.digikey.com/product-detail/en/samsung-electro-mechanics/CL10C150JB8NCNC/1276-2190-1-ND/3890276" H 1400 2150 60  0001 C CNN "Buy"
+F 4 "https://www.digikey.com/product-detail/en/yageo/CC0603JRNPO9BN150/311-1060-1-ND/302970" H 1400 2150 60  0001 C CNN "Buy"
 	1    1400 2150
 	0    1    1    0

Commit message: Removed the LV-Caps with the HV-Caps to remain consistent
Parts:
- C1, C35, C5: footprint Capacitor_SMD:C_0603_1608Metric -> Capacitor_SMD:C_0805_2012Metric; Buy https://www.digikey.com/product-detail/en/murata-electronics-north-america/GCM188R71C104KA37D/490-4774-1-ND/1641693 -> https://www.digikey.com/product-detail/en/murata-electronics-north-america/GCM21BR72A104KA37L/490-4789-1-ND/1641708
- C6: footprint (none) -> Capacitor_SMD:C_0805_2012Metric; Buy https://www.digikey.com/product-detail/en/murata-electronics-north-america/GCM188R71C104KA37D/490-4774-1-ND/1641693 -> https://www.digikey.com/product-detail/en/murata-electronics-north-america/GCM21BR72A104KA37L/490-4789-1-ND/1641708
- gave numbers to parts that had none: 5
Changed lines of the file:
@@
 F 0 "C1" H 860 1970 50  0000 L CNN
 F 1 "100nF" H 860 1820 50  0000 L CNN
-F 2 "Capacitor_SMD:C_0603_1608Metric" H 850 1900 50  0001 C CNN
+F 2 "Capacitor_SMD:C_0805_2012Metric" H 850 1900 50  0001 C CNN
 F 3 "" H 850 1900 50  0001 C CNN
-F 4 "https://www.digikey.com/product-detail/en/murata-electronics-north-america/GCM188R71C104KA37D/490-4774-1-ND/1641693" H 850 1900 50  0001 C CNN "Buy"
+F 4 "https://www.digikey.com/product-detail/en/murata-electronics-north-america/GCM21BR72A104KA37L/490-4789-1-ND/1641708" H 850 1900 50  0001 C CNN "Buy"
 	1    850  1900
 	1    0    0    -1
@@
 F 0 "C5" V 4100 1000 50  0000 L CNN
 F 1 "100nF" V 3900 950 50  0000 L CNN
-F 2 "Capacitor_SMD:C_0603_1608Metric" H 4000 1050 50  0001 C CNN
+F 2 "Capacitor_SMD:C_0805_2012Metric" H 4000 1050 50  0001 C CNN
 F 3 "" H 4000 1050 50  0001 C CNN
-F 4 "https://www.digikey.com/product-detail/en/murata-electronics-north-america/GCM188R71C104KA37D/490-4774-1-ND/1641693" V 4000 1050 50  0001 C CNN "Buy"
+F 4 "https://www.digikey.com/product-detail/en/murata-electronics-north-america/GCM21BR72A104KA37L/490-4789-1-ND/1641708" V 4000 1050 50  0001 C CNN "Buy"
 	1    4000 1050
 	0    1    1    0
@@
 F 0 "C6" H 7100 5975 50  0000 L CNN
 F 1 "100nF" H 7100 5825 50  0000 L CNN
-F 2 "" H 7075 5900 50  0001 C CNN
+F 2 "Capacitor_SMD:C_0805_2012Metric" H 7075 5900 50  0001 C CNN
 F 3 "~" H 7075 5900 50  0001 C CNN
-F 4 "https://www.digikey.com/product-detail/en/murata-electronics-north-america/GCM188R71C104KA37D/490-4774-1-ND/1641693" H 7075 5900 50  0001 C CNN "Buy"
+F 4 "https://www.digikey.com/product-detail/en/murata-electronics-north-america/GCM21BR72A104KA37L/490-4789-1-ND/1641708" H 7075 5900 50  0001 C CNN "Buy"
 	1    7075 5900
 	1    0    0    -1
@@
 F 0 "C35" V 4800 1000 50  0000 L CNN
 F 1 "100nF" V 4600 950 50  0000 L CNN
-F 2 "Capacitor_SMD:C_0603_1608Metric" H 4700 1050 50  0001 C CNN
+F 2 "Capacitor_SMD:C_0805_2012Metric" H 4700 1050 50  0001 C CNN
 F 3 "" H 4700 1050 50  0001 C CNN
-F 4 "https://www.digikey.com/product-detail/en/murata-electronics-north-america/GCM188R71C104KA37D/490-4774-1-ND/1641693" V 4700 1050 50  0001 C CNN "Buy"
+F 4 "https://www.digikey.com/product-detail/en/murata-electronics-north-america/GCM21BR72A104KA37L/490-4789-1-ND/1641708" V 4700 1050 50  0001 C CNN "Buy"
 	1    4700 1050
 	0    1    1    0
@@
 	2325 7500 2325 7025
 $Comp
-L connectors:RJ45-Dual J?
+L connectors:RJ45-Dual J11
 U 1 1 5ACE731B
 P 4325 6200
-F 0 "J?" H 4650 6600 60  0000 C CNN
+F 0 "J11" H 4650 6600 60  0000 C CNN
 F 1 "RJ45-Dual" H 4175 6600 60  0000 C CNN
 F 2 "" H 4275 6150 60  0001 C CNN
@@
 $EndComp
 $Comp
-L connectors:RJ45-Dual J?
+L connectors:RJ45-Dual J11
 U 2 1 5ACE7681
 P 5325 6200
-F 0 "J?" H 5650 6600 60  0000 C CNN
+F 0 "J11" H 5650 6600 60  0000 C CNN
 F 1 "RJ45-Dual" H 5175 6600 60  0000 C CNN
 F 2 "" H 5275 6150 60  0001 C CNN
@@
 $EndComp
 $Comp
-L connectors:RJ45-Dual J?
+L connectors:RJ45-Dual J2
 U 1 1 5AD02856
 P 1975 6200
-F 0 "J?" H 2300 6600 60  0000 C CNN
+F 0 "J2" H 2300 6600 60  0000 C CNN
 F 1 "RJ45-Dual" H 1825 6600 60  0000 C CNN
 F 2 "" H 1925 6150 60  0001 C CNN
@@
 $EndComp
 $Comp
-L connectors:RJ45-Dual J?
-U 1 1 5AD0285C
+L connectors:RJ45-Dual J2
+U 2 1 5AD0285C
 P 2975 6200
-F 0 "J?" H 3300 6600 60  0000 C CNN
+F 0 "J2" H 3300 6600 60  0000 C CNN
 F 1 "RJ45-Dual" H 2825 6600 60  0000 C CNN
 F 2 "" H 2925 6150 60  0001 C CNN
 F 3 "" H 2925 6150 60  0001 C CNN
-	1    2975 6200
-	1    0    0    -1
-$EndComp
-$Comp
-L power:GND #PWR?
+	2    2975 6200
+	1    0    0    -1
+$EndComp
+$Comp
+L power:GND #PWR0105
 U 1 1 5AD10161
 P 1475 6000
-F 0 "#PWR?" H 1475 5750 50  0001 C CNN
+F 0 "#PWR0105" H 1475 5750 50  0001 C CNN
 F 1 "GND" H 1480 5827 50  0000 C CNN
 F 2 "" H 1475 6000 50  0001 C CNN
@@
 OUT
 $Comp
-L Device:R R?
+L Device:R R8
 U 1 1 5AD83835
 P 850 1550
-F 0 "R?" V 930 1550 50  0000 C CNN
+F 0 "R8" V 930 1550 50  0000 C CNN
 F 1 "10k" V 850 1550 50  0000 C CNN
 F 2 "Resistor_SMD:R_0603_1608Metric" V 780 1550 50  0001 C CNN
@@
 $EndComp
 $Comp
-L power:+3.3V #PWR?
+L power:+3.3V #PWR0106
 U 1 1 5AD83C06
 P 850 1350
-F 0 "#PWR?" H 850 1200 50  0001 C CNN
+F 0 "#PWR0106" H 850 1200 50  0001 C CNN
 F 1 "+3.3V" H 850 1490 50  0000 C CNN
 F 2 "" H 850 1350 50  0001 C CNN
@@
 	850  1700 850  1750
 $Comp
-L Device:D_Small D?
+L Device:D_Small D3
 U 1 1 5AE82317
 P 1375 4100
-F 0 "D?" H 1375 4000 50  0000 C CNN
+F 0 "D3" H 1375 4000 50  0000 C CNN
 F 1 "D_Small" H 1375 4200 50  0000 C CNN
 F 2 "" V 1375 4100 50  0001 C CNN
@@
 	1275 4150 975  4150
 $Comp
-L Device:CP_Small C?
+L Device:CP_Small C36
 U 1 1 5AF930B2
 P 6825 5900
-F 0 "C?" H 6875 5975 50  0000 L CNN
+F 0 "C36" H 6875 5975 50  0000 L CNN
 F 1 "4.7μF" H 6850 5825 50  0000 L CNN
 F 2 "Capacitor_SMD:C_0603_1608Metric" H 6825 5900 50  0001 C CNN

Commit message: Replaced the 16V 1μF with a 25V-Version to use them on the 12V-Rail
Parts:
- C36, C4: value 4.7μF -> 1μF; footprint Capacitor_SMD:C_0603_1608Metric -> Capacitor_SMD:C_0805_2012Metric; symbol Device:CP_Small -> Device:C_Small; Digikey (none) -> https://www.digikey.com/product-detail/en/taiyo-yuden/TMK21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
Changed lines of the file:
@@
 $EndComp
 $Comp
-L Device:CP_Small C4
+L Device:C_Small C4
 U 1 1 5A469943
 P 4000 775
 F 0 "C4" V 4100 725 50  0000 L CNN
-F 1 "4.7μF" V 3900 675 50  0000 L CNN
-F 2 "Capacitor_SMD:C_0603_1608Metric" H 4000 775 50  0001 C CNN
+F 1 "1μF" V 3900 725 50  0000 L CNN
+F 2 "Capacitor_SMD:C_0805_2012Metric" H 4000 775 50  0001 C CNN
 F 3 "" H 4000 775 50  0001 C CNN
+F 4 "https://www.digikey.com/product-detail/en/taiyo-yuden/TMK212B7105MG-T/587-5595-1-ND/7067270" V 4000 775 50  0001 C CNN "Digikey"
 	1    4000 775
 	0    1    1    0
@@
 	1275 4150 975  4150
 $Comp
-L Device:CP_Small C36
+L Device:C_Small C36
 U 1 1 5AF930B2
 P 6825 5900
-F 0 "C36" H 6875 5975 50  0000 L CNN
-F 1 "4.7μF" H 6850 5825 50  0000 L CNN
-F 2 "Capacitor_SMD:C_0603_1608Metric" H 6825 5900 50  0001 C CNN
+F 0 "C36" H 6825 5975 50  0000 L CNN
+F 1 "1μF" H 6825 5825 50  0000 L CNN
+F 2 "Capacitor_SMD:C_0805_2012Metric" H 6825 5900 50  0001 C CNN
 F 3 "" H 6825 5900 50  0001 C CNN
+F 4 "https://www.digikey.com/product-detail/en/taiyo-yuden/TMK212B7105MG-T/587-5595-1-ND/7067270" H 6825 5900 50  0001 C CNN "Digikey"
 	1    6825 5900
 	1    0    0    -1

Commit message: Replaced the Digikey-Field with a Buy-Field
Parts:
- C36, C4: Buy (none) -> https://www.digikey.com/product-detail/en/taiyo-yuden/TMK21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; Digikey https://www.digikey.com/product-detail/en/taiyo-yuden/TMK21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 -> (none)
Changed lines of the file:
@@
 F 2 "Capacitor_SMD:C_0805_2012Metric" H 4000 775 50  0001 C CNN
 F 3 "" H 4000 775 50  0001 C CNN
-F 4 "https://www.digikey.com/product-detail/en/taiyo-yuden/TMK212B7105MG-T/587-5595-1-ND/7067270" V 4000 775 50  0001 C CNN "Digikey"
+F 4 "https://www.digikey.com/product-detail/en/taiyo-yuden/TMK212B7105MG-T/587-5595-1-ND/7067270" V 4000 775 50  0001 C CNN "Buy"
 	1    4000 775
 	0    1    1    0
@@
 F 2 "Capacitor_SMD:C_0805_2012Metric" H 6825 5900 50  0001 C CNN
 F 3 "" H 6825 5900 50  0001 C CNN
-F 4 "https://www.digikey.com/product-detail/en/taiyo-yuden/TMK212B7105MG-T/587-5595-1-ND/7067270" H 6825 5900 50  0001 C CNN "Digikey"
+F 4 "https://www.digikey.com/product-detail/en/taiyo-yuden/TMK212B7105MG-T/587-5595-1-ND/7067270" H 6825 5900 50  0001 C CNN "Buy"
 	1    6825 5900
 	1    0    0    -1
