File: Panel.sch (KiCad schematic (older format))
At the start: 10 parts, among them J6 Rotated_Barrel, U7 LM3406HV

Commit message: Footprint-Association: 90%
Parts:
- J7: renamed from J6; footprint (none) -> Connectors:BARREL_JACK
- U7: footprint (none) -> Housings_SSOP:TSSOP-14_4.4x5mm_Pitch0.65mm
Changed lines of the file:
@@
 AR Path="/5A4C34AF/5A7753B7" Ref="R13"  Part="1"
 AR Path="/5A4C3F5F/5A7753B7" Ref="R15"  Part="1"
-F 0 "R15" V 1430 1300 50  0000 C CNN
+F 0 "R13" V 1430 1300 50  0000 C CNN
 F 1 "162k" V 1350 1300 50  0000 C CNN
 F 2 "Resistors_SMD:R_0603" V 1280 1300 50  0001 C CNN
@@
 AR Path="/5A4C34AF/5A77745B" Ref="C22"  Part="1"
 AR Path="/5A4C3F5F/5A77745B" Ref="C26"  Part="1"
-F 0 "C26" H 1510 2220 50  0000 L CNN
+F 0 "C22" H 1510 2220 50  0000 L CNN
 F 1 "100nF" H 1510 2070 50  0000 L CNN
 F 2 "Capacitors_SMD:C_0603" H 1500 2150 50  0001 C CNN
@@
 $EndComp
 $Comp
-L GND #PWR58
+L GND #PWR061
 U 1 1 5A777BDD
 P 1500 2300
-AR Path="/5A4C34AF/5A777BDD" Ref="#PWR58"  Part="1"
-AR Path="/5A4C3F5F/5A777BDD" Ref="#PWR65"  Part="1"
-F 0 "#PWR65" H 1500 2050 50  0001 C CNN
+AR Path="/5A4C34AF/5A777BDD" Ref="#PWR061"  Part="1"
+AR Path="/5A4C3F5F/5A777BDD" Ref="#PWR068"  Part="1"
+F 0 "#PWR061" H 1500 2050 50  0001 C CNN
 F 1 "GND" H 1500 2150 50  0000 C CNN
 F 2 "" H 1500 2300 50  0001 C CNN
@@
 AR Path="/5A4C34AF/5A777CD4" Ref="C23"  Part="1"
 AR Path="/5A4C3F5F/5A777CD4" Ref="C27"  Part="1"
-F 0 "C27" H 2710 2220 50  0000 L CNN
+F 0 "C23" H 2710 2220 50  0000 L CNN
 F 1 "100nF" H 2710 2070 50  0000 L CNN
 F 2 "Capacitors_SMD:C_0603" H 2700 2150 50  0001 C CNN
@@
 $EndComp
 $Comp
-L GND #PWR60
+L GND #PWR062
 U 1 1 5A777CDA
 P 2700 2300
-AR Path="/5A4C34AF/5A777CDA" Ref="#PWR60"  Part="1"
-AR Path="/5A4C3F5F/5A777CDA" Ref="#PWR67"  Part="1"
-F 0 "#PWR67" H 2700 2050 50  0001 C CNN
+AR Path="/5A4C34AF/5A777CDA" Ref="#PWR062"  Part="1"
+AR Path="/5A4C3F5F/5A777CDA" Ref="#PWR069"  Part="1"
+F 0 "#PWR062" H 2700 2050 50  0001 C CNN
 F 1 "GND" H 2700 2150 50  0000 C CNN
 F 2 "" H 2700 2300 50  0001 C CNN
@@
 $EndComp
 $Comp
-L GND #PWR59
+L GND #PWR063
 U 1 1 5A777FA3
 P 2100 2300
-AR Path="/5A4C34AF/5A777FA3" Ref="#PWR59"  Part="1"
-AR Path="/5A4C3F5F/5A777FA3" Ref="#PWR66"  Part="1"
-F 0 "#PWR66" H 2100 2050 50  0001 C CNN
+AR Path="/5A4C34AF/5A777FA3" Ref="#PWR063"  Part="1"
+AR Path="/5A4C3F5F/5A777FA3" Ref="#PWR070"  Part="1"
+F 0 "#PWR063" H 2100 2050 50  0001 C CNN
 F 1 "GND" H 2100 2150 50  0000 C CNN
 F 2 "" H 2100 2300 50  0001 C CNN
@@
 AR Path="/5A4C34AF/5A77816D" Ref="C20"  Part="1"
 AR Path="/5A4C3F5F/5A77816D" Ref="C24"  Part="1"
-F 0 "C24" H 2460 920 50  0000 L CNN
+F 0 "C20" H 2460 920 50  0000 L CNN
 F 1 "22nF" H 2460 770 50  0000 L CNN
 F 2 "Capacitors_SMD:C_0603" H 2450 850 50  0001 C CNN
@@
 AR Path="/5A4C34AF/5A77899A" Ref="L3"  Part="1"
 AR Path="/5A4C3F5F/5A77899A" Ref="L4"  Part="1"
-F 0 "L4" V 3200 1050 50  0000 C CNN
+F 0 "L3" V 3200 1050 50  0000 C CNN
 F 1 "33μH" V 3325 1050 50  0000 C CNN
 F 2 "" H 3250 1050 50  0001 C CNN
@@
 AR Path="/5A4C34AF/5A7789F9" Ref="D1"  Part="1"
 AR Path="/5A4C3F5F/5A7789F9" Ref="D2"  Part="1"
-F 0 "D2" H 3000 1400 50  0000 C CNN
+F 0 "D1" H 3000 1400 50  0000 C CNN
 F 1 "D_Schot" H 2950 1200 50  0000 C CNN
 F 2 "Diodes_SMD:D_SOD-123" H 3000 1300 50  0001 C CNN
@@
 Connection ~ 3000 1050
 $Comp
-L GND #PWR61
+L GND #PWR064
 U 1 1 5A778B62
 P 3000 2300
-AR Path="/5A4C34AF/5A778B62" Ref="#PWR61"  Part="1"
-AR Path="/5A4C3F5F/5A778B62" Ref="#PWR68"  Part="1"
-F 0 "#PWR68" H 3000 2050 50  0001 C CNN
+AR Path="/5A4C34AF/5A778B62" Ref="#PWR064"  Part="1"
+AR Path="/5A4C3F5F/5A778B62" Ref="#PWR071"  Part="1"
+F 0 "#PWR064" H 3000 2050 50  0001 C CNN
 F 1 "GND" H 3000 2150 50  0000 C CNN
 F 2 "" H 3000 2300 50  0001 C CNN
@@
 	3000 2300 3000 1450
 $Comp
-L Rotated_Barrel J6
+L Rotated_Barrel J7
 U 1 1 5A779AD3
 P 3700 1500
-AR Path="/5A4C34AF/5A779AD3" Ref="J6"  Part="1"
-AR Path="/5A4C3F5F/5A779AD3" Ref="J7"  Part="1"
+AR Path="/5A4C34AF/5A779AD3" Ref="J7"  Part="1"
+AR Path="/5A4C3F5F/5A779AD3" Ref="J8"  Part="1"
 F 0 "J7" H 3700 1710 50  0000 C CNN
 F 1 "Rotated_Barrel" H 3750 1350 50  0000 C CNN
-F 2 "" H 3750 1440 50  0001 C CNN
+F 2 "Connectors:BARREL_JACK" H 3750 1440 50  0001 C CNN
 F 3 "" H 3750 1440 50  0001 C CNN
 	1    3700 1500
@@
 AR Path="/5A4C34AF/5A77A2E1" Ref="R14"  Part="1"
 AR Path="/5A4C3F5F/5A77A2E1" Ref="R16"  Part="1"
-F 0 "R16" V 3530 1900 50  0000 C CNN
+F 0 "R14" V 3530 1900 50  0000 C CNN
 F 1 "0R16" V 3450 1900 50  0000 C CNN
 F 2 "Resistors_SMD:R_0603" V 3380 1900 50  0001 C CNN
@@
 Connection ~ 3450 1700
 $Comp
-L GND #PWR62
+L GND #PWR065
 U 1 1 5A77A9CB
 P 3450 2300
-AR Path="/5A4C34AF/5A77A9CB" Ref="#PWR62"  Part="1"
-AR Path="/5A4C3F5F/5A77A9CB" Ref="#PWR69"  Part="1"
-F 0 "#PWR69" H 3450 2050 50  0001 C CNN
+AR Path="/5A4C34AF/5A77A9CB" Ref="#PWR065"  Part="1"
+AR Path="/5A4C3F5F/5A77A9CB" Ref="#PWR072"  Part="1"
+F 0 "#PWR065" H 3450 2050 50  0001 C CNN
 F 1 "GND" H 3450 2150 50  0000 C CNN
 F 2 "" H 3450 2300 50  0001 C CNN
@@
 AR Path="/5A4C34AF/5A77D10E" Ref="C21"  Part="1"
 AR Path="/5A4C3F5F/5A77D10E" Ref="C25"  Part="1"
-F 0 "C25" H 1110 1370 50  0000 L CNN
+F 0 "C21" H 1110 1370 50  0000 L CNN
 F 1 "1μF" H 1110 1220 50  0000 L CNN
 F 2 "Capacitors_SMD:C_0603" H 1100 1300 50  0001 C CNN
@@
 Connection ~ 1100 1050
 $Comp
-L GND #PWR57
+L GND #PWR066
 U 1 1 5A77D43C
 P 1100 2300
-AR Path="/5A4C34AF/5A77D43C" Ref="#PWR57"  Part="1"
-AR Path="/5A4C3F5F/5A77D43C" Ref="#PWR64"  Part="1"
-F 0 "#PWR64" H 1100 2050 50  0001 C CNN
+AR Path="/5A4C34AF/5A77D43C" Ref="#PWR066"  Part="1"
+AR Path="/5A4C3F5F/5A77D43C" Ref="#PWR073"  Part="1"
+F 0 "#PWR066" H 1100 2050 50  0001 C CNN
 F 1 "GND" H 1100 2150 50  0000 C CNN
 F 2 "" H 1100 2300 50  0001 C CNN
@@
 AR Path="/5A4C34AF/5A77E620" Ref="U7"  Part="1"
 AR Path="/5A4C3F5F/5A77E620" Ref="U8"  Part="1"
-F 0 "U8" H 2500 950 60  0000 C CNN
+F 0 "U7" H 2500 950 60  0000 C CNN
 F 1 "LM3406HV" H 1900 2050 60  0000 C CNN
-F 2 "" H 2100 2100 60  0001 C CNN
+F 2 "Housings_SSOP:TSSOP-14_4.4x5mm_Pitch0.65mm" H 2100 2100 60  0001 C CNN
 F 3 "http://www.ti.com/lit/ds/symlink/lm3406.pdf" H 2100 2100 60  0001 C CNN
 F 4 "https://www.digikey.com/product-detail/en/texas-instruments/LM3406HVMHX-NOPB/LM3406HVMHX-NOPBCT-ND/3526958" H 2100 1500 60  0001 C CNN "Digikey"
@@
 	4100 475  4100 2500
 $Comp
-L +48V #PWR56
+L +48V #PWR067
 U 1 1 5A84C99A
 P 1050 950
-AR Path="/5A4C34AF/5A84C99A" Ref="#PWR56"  Part="1"
-AR Path="/5A4C3F5F/5A84C99A" Ref="#PWR63"  Part="1"
-F 0 "#PWR63" H 1050 800 50  0001 C CNN
+AR Path="/5A4C34AF/5A84C99A" Ref="#PWR067"  Part="1"
+AR Path="/5A4C3F5F/5A84C99A" Ref="#PWR074"  Part="1"
+F 0 "#PWR067" H 1050 800 50  0001 C CNN
 F 1 "+48V" H 1050 1090 50  0000 C CNN
 F 2 "" H 1050 950 50  0001 C CNN

Commit message: Changed the 5V-Regulator
Parts:
- C20, C21, C22, C23: symbol C_Small -> device:C_Small
- D1: symbol D_Schottky -> device:D_Schottky
- J7: symbol Rotated_Barrel -> jacks:Rotated_Barrel
- L3: symbol L -> device:L
- R13, R14: symbol R -> device:R
- U7: symbol LM3406HV -> ledDriver:LM3406HV
Changed lines of the file:
@@
-EESchema Schematic File Version 2
-LIBS:power
-LIBS:device
-LIBS:switches
-LIBS:transistors
-LIBS:conn
-LIBS:linear
-LIBS:regul
-LIBS:74xx
-LIBS:analog_switches
-LIBS:texas
-LIBS:interface
-LIBS:philips
-LIBS:cypress
-LIBS:siliconi
-LIBS:opto
-LIBS:contrib
-LIBS:stm32s
-LIBS:transceiver
-LIBS:switchingR
-LIBS:ledDriver
-LIBS:jacks
-LIBS:sensors
+EESchema Schematic File Version 4
 LIBS:Hardware-cache
-EELAYER 25 0
+EELAYER 26 0
 EELAYER END
 $Descr A4 11693 8268
@@
 $EndDescr
 $Comp
-L R R13
+L device:R R13
 U 1 1 5A7753B7
 P 1350 1300
@@
 $EndComp
 $Comp
-L C_Small C22
+L device:C_Small C22
 U 1 1 5A77745B
 P 1500 2150
@@
 $EndComp
 $Comp
-L GND #PWR061
+L power:GND #PWR061
 U 1 1 5A777BDD
 P 1500 2300
@@
 $EndComp
 $Comp
-L C_Small C23
+L device:C_Small C23
 U 1 1 5A777CD4
 P 2700 2150
@@
 $EndComp
 $Comp
-L GND #PWR062
+L power:GND #PWR062
 U 1 1 5A777CDA
 P 2700 2300
@@
 $EndComp
 $Comp
-L GND #PWR063
+L power:GND #PWR063
 U 1 1 5A777FA3
 P 2100 2300
@@
 $EndComp
 $Comp
-L C_Small C20
+L device:C_Small C20
 U 1 1 5A77816D
 P 2450 850
@@
 Connection ~ 2700 1050
 $Comp
-L L L3
+L device:L L3
 U 1 1 5A77899A
 P 3250 1050
@@
 $EndComp
 $Comp
-L D_Schottky D1
+L device:D_Schottky D1
 U 1 1 5A7789F9
 P 3000 1300
@@
 Connection ~ 3000 1050
 $Comp
-L GND #PWR064
+L power:GND #PWR064
 U 1 1 5A778B62
 P 3000 2300
@@
 	3000 2300 3000 1450
 $Comp
-L Rotated_Barrel J7
+L jacks:Rotated_Barrel J7
 U 1 1 5A779AD3
 P 3700 1500
@@
 Connection ~ 3450 1400
 $Comp
-L R R14
+L device:R R14
 U 1 1 5A77A2E1
 P 3450 1900
@@
 Connection ~ 3450 1700
 $Comp
-L GND #PWR065
+L power:GND #PWR065
 U 1 1 5A77A9CB
 P 3450 2300
@@
 	3450 2300 3450 2050
 $Comp
-L C_Small C21
+L device:C_Small C21
 U 1 1 5A77D10E
 P 1100 1300
@@
 Connection ~ 1100 1050
 $Comp
-L GND #PWR066
+L power:GND #PWR066
 U 1 1 5A77D43C
 P 1100 2300
@@
 	1000 1700 1550 1700
 $Comp
-L LM3406HV U7
+L ledDriver:LM3406HV U7
 U 1 1 5A77E620
 P 2100 1500
@@
 	4100 475  4100 2500
 $Comp
-L +48V #PWR067
+L power:+48V #PWR067
 U 1 1 5A84C99A
 P 1050 950

Commit message: Minor Bugfixes
Connections:
- wire segments 34 -> 44
Changed lines of the file:
@@
 $Descr A4 11693 8268
 encoding utf-8
-Sheet 4 7
+Sheet 3 7
 Title ""
 Date "2018-02-14"
@@
 	1500 1250 1550 1250
 Wire Wire Line
-	1500 1050 1500 1250
+	1500 1050 1500 1150
 Wire Wire Line
 	1500 1150 1550 1150
 Connection ~ 1500 1150
 Wire Wire Line
-	1050 1050 1550 1050
+	1050 1050 1100 1050
 Connection ~ 1500 1050
 Wire Wire Line
@@
 	2550 850  2700 850
 Wire Wire Line
-	2650 1050 3100 1050
-Wire Wire Line
-	2700 850  2700 1150
+	2650 1050 2700 1050
+Wire Wire Line
+	2700 850  2700 1050
 Wire Wire Line
 	1350 1500 1350 1450
@@
 	3450 1050 3450 1400
 Wire Wire Line
-	2650 1400 3500 1400
+	2650 1400 3450 1400
 Connection ~ 3450 1400
 $Comp
@@
 $EndComp
 Wire Wire Line
-	3450 1500 3450 1750
+	3450 1500 3450 1600
 Wire Wire Line
 	3450 1500 3500 1500
@@
 Wire Notes Line
 	4100 2500 475  2500
+Wire Wire Line
+	1500 1150 1500 1250
+Wire Wire Line
+	1500 1050 1550 1050
+Wire Wire Line
+	1350 1050 1500 1050
+Wire Wire Line
+	2700 1050 3000 1050
+Wire Wire Line
+	2700 1050 2700 1150
+Wire Wire Line
+	3000 1050 3100 1050
+Wire Wire Line
+	3450 1400 3500 1400
+Wire Wire Line
+	3450 1600 3450 1700
+Wire Wire Line
+	3450 1700 3450 1750
+Wire Wire Line
+	1100 1050 1350 1050
 $EndSCHEMATC

Commit message: Updated to the new libraries
Parts:
- C20: renamed from C21; symbol device:C_Small -> Device:C_Small
- C21: renamed from C22; symbol device:C_Small -> Device:C_Small
- C22: renamed from C20; symbol device:C_Small -> Device:C_Small
- C23: symbol device:C_Small -> Device:C_Small
- D1: symbol device:D_Schottky -> Device:D_Schottky
- L3: symbol device:L -> Device:L
- R11: renamed from R13; symbol device:R -> Device:R
- R12: renamed from R14; symbol device:R -> Device:R
Changed lines of the file:
@@
 $EndDescr
 $Comp
-L device:R R13
+L Device:R R11
 U 1 1 5A7753B7
 P 1350 1300
-AR Path="/5A4C34AF/5A7753B7" Ref="R13"  Part="1"
-AR Path="/5A4C3F5F/5A7753B7" Ref="R15"  Part="1"
+AR Path="/5A4C34AF/5A7753B7" Ref="R11"  Part="1"
+AR Path="/5A4C3F5F/5A7753B7" Ref="R13"  Part="1"
 F 0 "R13" V 1430 1300 50  0000 C CNN
 F 1 "162k" V 1350 1300 50  0000 C CNN
@@
 $EndComp
 $Comp
-L device:C_Small C22
+L Device:C_Small C21
 U 1 1 5A77745B
 P 1500 2150
-AR Path="/5A4C34AF/5A77745B" Ref="C22"  Part="1"
-AR Path="/5A4C3F5F/5A77745B" Ref="C26"  Part="1"
-F 0 "C22" H 1510 2220 50  0000 L CNN
+AR Path="/5A4C34AF/5A77745B" Ref="C21"  Part="1"
+AR Path="/5A4C3F5F/5A77745B" Ref="C25"  Part="1"
+F 0 "C25" H 1510 2220 50  0000 L CNN
 F 1 "100nF" H 1510 2070 50  0000 L CNN
 F 2 "Capacitors_SMD:C_0603" H 1500 2150 50  0001 C CNN
@@
 $EndComp
 $Comp
-L power:GND #PWR061
+L power:GND #PWR058
 U 1 1 5A777BDD
 P 1500 2300
-AR Path="/5A4C34AF/5A777BDD" Ref="#PWR061"  Part="1"
-AR Path="/5A4C3F5F/5A777BDD" Ref="#PWR068"  Part="1"
-F 0 "#PWR061" H 1500 2050 50  0001 C CNN
+AR Path="/5A4C34AF/5A777BDD" Ref="#PWR058"  Part="1"
+AR Path="/5A4C3F5F/5A777BDD" Ref="#PWR065"  Part="1"
+F 0 "#PWR065" H 1500 2050 50  0001 C CNN
 F 1 "GND" H 1500 2150 50  0000 C CNN
 F 2 "" H 1500 2300 50  0001 C CNN
@@
 $EndComp
 $Comp
-L device:C_Small C23
+L Device:C_Small C23
 U 1 1 5A777CD4
 P 2700 2150
 AR Path="/5A4C34AF/5A777CD4" Ref="C23"  Part="1"
 AR Path="/5A4C3F5F/5A777CD4" Ref="C27"  Part="1"
-F 0 "C23" H 2710 2220 50  0000 L CNN
+F 0 "C27" H 2710 2220 50  0000 L CNN
 F 1 "100nF" H 2710 2070 50  0000 L CNN
 F 2 "Capacitors_SMD:C_0603" H 2700 2150 50  0001 C CNN
@@
 $EndComp
 $Comp
-L power:GND #PWR062
+L power:GND #PWR060
 U 1 1 5A777CDA
 P 2700 2300
-AR Path="/5A4C34AF/5A777CDA" Ref="#PWR062"  Part="1"
-AR Path="/5A4C3F5F/5A777CDA" Ref="#PWR069"  Part="1"
-F 0 "#PWR062" H 2700 2050 50  0001 C CNN
+AR Path="/5A4C34AF/5A777CDA" Ref="#PWR060"  Part="1"
+AR Path="/5A4C3F5F/5A777CDA" Ref="#PWR067"  Part="1"
+F 0 "#PWR067" H 2700 2050 50  0001 C CNN
 F 1 "GND" H 2700 2150 50  0000 C CNN
 F 2 "" H 2700 2300 50  0001 C CNN
@@
 $EndComp
 $Comp
-L power:GND #PWR063
+L power:GND #PWR059
 U 1 1 5A777FA3
 P 2100 2300
-AR Path="/5A4C34AF/5A777FA3" Ref="#PWR063"  Part="1"
-AR Path="/5A4C3F5F/5A777FA3" Ref="#PWR070"  Part="1"
-F 0 "#PWR063" H 2100 2050 50  0001 C CNN
+AR Path="/5A4C34AF/5A777FA3" Ref="#PWR059"  Part="1"
+AR Path="/5A4C3F5F/5A777FA3" Ref="#PWR066"  Part="1"
+F 0 "#PWR066" H 2100 2050 50  0001 C CNN
 F 1 "GND" H 2100 2150 50  0000 C CNN
 F 2 "" H 2100 2300 50  0001 C CNN
@@
 $EndComp
 $Comp
-L device:C_Small C20
+L Device:C_Small C22
 U 1 1 5A77816D
 P 2450 850
-AR Path="/5A4C34AF/5A77816D" Ref="C20"  Part="1"
-AR Path="/5A4C3F5F/5A77816D" Ref="C24"  Part="1"
-F 0 "C20" H 2460 920 50  0000 L CNN
+AR Path="/5A4C34AF/5A77816D" Ref="C22"  Part="1"
+AR Path="/5A4C3F5F/5A77816D" Ref="C26"  Part="1"
+F 0 "C26" H 2460 920 50  0000 L CNN
 F 1 "22nF" H 2460 770 50  0000 L CNN
 F 2 "Capacitors_SMD:C_0603" H 2450 850 50  0001 C CNN
@@
 Connection ~ 2700 1050
 $Comp
-L device:L L3
+L Device:L L3
 U 1 1 5A77899A
 P 3250 1050
 AR Path="/5A4C34AF/5A77899A" Ref="L3"  Part="1"
 AR Path="/5A4C3F5F/5A77899A" Ref="L4"  Part="1"
-F 0 "L3" V 3200 1050 50  0000 C CNN
+F 0 "L4" V 3200 1050 50  0000 C CNN
 F 1 "33μH" V 3325 1050 50  0000 C CNN
 F 2 "" H 3250 1050 50  0001 C CNN
@@
 $EndComp
 $Comp
-L device:D_Schottky D1
+L Device:D_Schottky D1
 U 1 1 5A7789F9
 P 3000 1300
 AR Path="/5A4C34AF/5A7789F9" Ref="D1"  Part="1"
 AR Path="/5A4C3F5F/5A7789F9" Ref="D2"  Part="1"
-F 0 "D1" H 3000 1400 50  0000 C CNN
+F 0 "D2" H 3000 1400 50  0000 C CNN
 F 1 "D_Schot" H 2950 1200 50  0000 C CNN
 F 2 "Diodes_SMD:D_SOD-123" H 3000 1300 50  0001 C CNN
@@
 Connection ~ 3000 1050
 $Comp
-L power:GND #PWR064
+L power:GND #PWR061
 U 1 1 5A778B62
 P 3000 2300
-AR Path="/5A4C34AF/5A778B62" Ref="#PWR064"  Part="1"
-AR Path="/5A4C3F5F/5A778B62" Ref="#PWR071"  Part="1"
-F 0 "#PWR064" H 3000 2050 50  0001 C CNN
+AR Path="/5A4C34AF/5A778B62" Ref="#PWR061"  Part="1"
+AR Path="/5A4C3F5F/5A778B62" Ref="#PWR068"  Part="1"
+F 0 "#PWR068" H 3000 2050 50  0001 C CNN
 F 1 "GND" H 3000 2150 50  0000 C CNN
 F 2 "" H 3000 2300 50  0001 C CNN
@@
 AR Path="/5A4C34AF/5A779AD3" Ref="J7"  Part="1"
 AR Path="/5A4C3F5F/5A779AD3" Ref="J8"  Part="1"
-F 0 "J7" H 3700 1710 50  0000 C CNN
+F 0 "J8" H 3700 1710 50  0000 C CNN
 F 1 "Rotated_Barrel" H 3750 1350 50  0000 C CNN
 F 2 "Connectors:BARREL_JACK" H 3750 1440 50  0001 C CNN
@@
 Connection ~ 3450 1400
 $Comp
-L device:R R14
+L Device:R R12
 U 1 1 5A77A2E1
 P 3450 1900
-AR Path="/5A4C34AF/5A77A2E1" Ref="R14"  Part="1"
-AR Path="/5A4C3F5F/5A77A2E1" Ref="R16"  Part="1"
+AR Path="/5A4C34AF/5A77A2E1" Ref="R12"  Part="1"
+AR Path="/5A4C3F5F/5A77A2E1" Ref="R14"  Part="1"
 F 0 "R14" V 3530 1900 50  0000 C CNN
 F 1 "0R16" V 3450 1900 50  0000 C CNN
@@
 Connection ~ 3450 1700
 $Comp
-L power:GND #PWR065
+L power:GND #PWR062
 U 1 1 5A77A9CB
 P 3450 2300
-AR Path="/5A4C34AF/5A77A9CB" Ref="#PWR065"  Part="1"
-AR Path="/5A4C3F5F/5A77A9CB" Ref="#PWR072"  Part="1"
-F 0 "#PWR065" H 3450 2050 50  0001 C CNN
+AR Path="/5A4C34AF/5A77A9CB" Ref="#PWR062"  Part="1"
+AR Path="/5A4C3F5F/5A77A9CB" Ref="#PWR069"  Part="1"
+F 0 "#PWR069" H 3450 2050 50  0001 C CNN
 F 1 "GND" H 3450 2150 50  0000 C CNN
 F 2 "" H 3450 2300 50  0001 C CNN
@@
 	3450 2300 3450 2050
 $Comp
-L device:C_Small C21
+L Device:C_Small C20
 U 1 1 5A77D10E
 P 1100 1300
-AR Path="/5A4C34AF/5A77D10E" Ref="C21"  Part="1"
-AR Path="/5A4C3F5F/5A77D10E" Ref="C25"  Part="1"
-F 0 "C21" H 1110 1370 50  0000 L CNN
+AR Path="/5A4C34AF/5A77D10E" Ref="C20"  Part="1"
+AR Path="/5A4C3F5F/5A77D10E" Ref="C24"  Part="1"
+F 0 "C24" H 1110 1370 50  0000 L CNN
 F 1 "1μF" H 1110 1220 50  0000 L CNN
 F 2 "Capacitors_SMD:C_0603" H 1100 1300 50  0001 C CNN
@@
 Connection ~ 1100 1050
 $Comp
-L power:GND #PWR066
+L power:GND #PWR057
 U 1 1 5A77D43C
 P 1100 2300
-AR Path="/5A4C34AF/5A77D43C" Ref="#PWR066"  Part="1"
-AR Path="/5A4C3F5F/5A77D43C" Ref="#PWR073"  Part="1"
-F 0 "#PWR066" H 1100 2050 50  0001 C CNN
+AR Path="/5A4C34AF/5A77D43C" Ref="#PWR057"  Part="1"
+AR Path="/5A4C3F5F/5A77D43C" Ref="#PWR064"  Part="1"
+F 0 "#PWR064" H 1100 2050 50  0001 C CNN
 F 1 "GND" H 1100 2150 50  0000 C CNN
 F 2 "" H 1100 2300 50  0001 C CNN
@@
 AR Path="/5A4C34AF/5A77E620" Ref="U7"  Part="1"
 AR Path="/5A4C3F5F/5A77E620" Ref="U8"  Part="1"
-F 0 "U7" H 2500 950 60  0000 C CNN
+F 0 "U8" H 2500 950 60  0000 C CNN
 F 1 "LM3406HV" H 1900 2050 60  0000 C CNN
 F 2 "Housings_SSOP:TSSOP-14_4.4x5mm_Pitch0.65mm" H 2100 2100 60  0001 C CNN
@@
 	4100 475  4100 2500
 $Comp
-L power:+48V #PWR067
+L power:+48V #PWR056
 U 1 1 5A84C99A
 P 1050 950
-AR Path="/5A4C34AF/5A84C99A" Ref="#PWR067"  Part="1"
-AR Path="/5A4C3F5F/5A84C99A" Ref="#PWR074"  Part="1"
-F 0 "#PWR067" H 1050 800 50  0001 C CNN
+AR Path="/5A4C34AF/5A84C99A" Ref="#PWR056"  Part="1"
+AR Path="/5A4C3F5F/5A84C99A" Ref="#PWR063"  Part="1"
+F 0 "#PWR063" H 1050 800 50  0001 C CNN
 F 1 "+48V" H 1050 1090 50  0000 C CNN
 F 2 "" H 1050 950 50  0001 C CNN

Commit message: Renamed jacks to connectors
Parts:
- J7: symbol jacks:Rotated_Barrel -> connectors:Rotated_Barrel
Changed lines of the file:
@@
 	3000 2300 3000 1450
 $Comp
-L jacks:Rotated_Barrel J7
+L connectors:Rotated_Barrel J7
 U 1 1 5A779AD3
 P 3700 1500

Commit message: Changed the RJ45 to a Quad-Type
Parts:
- renumbered J7 to J6
Changed lines of the file:
@@
 $EndComp
 $Comp
-L power:GND #PWR058
+L power:GND #PWR061
 U 1 1 5A777BDD
 P 1500 2300
-AR Path="/5A4C34AF/5A777BDD" Ref="#PWR058"  Part="1"
-AR Path="/5A4C3F5F/5A777BDD" Ref="#PWR065"  Part="1"
-F 0 "#PWR065" H 1500 2050 50  0001 C CNN
+AR Path="/5A4C34AF/5A777BDD" Ref="#PWR061"  Part="1"
+AR Path="/5A4C3F5F/5A777BDD" Ref="#PWR068"  Part="1"
+F 0 "#PWR068" H 1500 2050 50  0001 C CNN
 F 1 "GND" H 1500 2150 50  0000 C CNN
 F 2 "" H 1500 2300 50  0001 C CNN
@@
 $EndComp
 $Comp
-L power:GND #PWR060
+L power:GND #PWR063
 U 1 1 5A777CDA
 P 2700 2300
-AR Path="/5A4C34AF/5A777CDA" Ref="#PWR060"  Part="1"
-AR Path="/5A4C3F5F/5A777CDA" Ref="#PWR067"  Part="1"
-F 0 "#PWR067" H 2700 2050 50  0001 C CNN
+AR Path="/5A4C34AF/5A777CDA" Ref="#PWR063"  Part="1"
+AR Path="/5A4C3F5F/5A777CDA" Ref="#PWR070"  Part="1"
+F 0 "#PWR070" H 2700 2050 50  0001 C CNN
 F 1 "GND" H 2700 2150 50  0000 C CNN
 F 2 "" H 2700 2300 50  0001 C CNN
@@
 $EndComp
 $Comp
-L power:GND #PWR059
+L power:GND #PWR062
 U 1 1 5A777FA3
 P 2100 2300
-AR Path="/5A4C34AF/5A777FA3" Ref="#PWR059"  Part="1"
-AR Path="/5A4C3F5F/5A777FA3" Ref="#PWR066"  Part="1"
-F 0 "#PWR066" H 2100 2050 50  0001 C CNN
+AR Path="/5A4C34AF/5A777FA3" Ref="#PWR062"  Part="1"
+AR Path="/5A4C3F5F/5A777FA3" Ref="#PWR069"  Part="1"
+F 0 "#PWR069" H 2100 2050 50  0001 C CNN
 F 1 "GND" H 2100 2150 50  0000 C CNN
 F 2 "" H 2100 2300 50  0001 C CNN
@@
 Connection ~ 3000 1050
 $Comp
-L power:GND #PWR061
+L power:GND #PWR064
 U 1 1 5A778B62
 P 3000 2300
-AR Path="/5A4C34AF/5A778B62" Ref="#PWR061"  Part="1"
-AR Path="/5A4C3F5F/5A778B62" Ref="#PWR068"  Part="1"
-F 0 "#PWR068" H 3000 2050 50  0001 C CNN
+AR Path="/5A4C34AF/5A778B62" Ref="#PWR064"  Part="1"
+AR Path="/5A4C3F5F/5A778B62" Ref="#PWR071"  Part="1"
+F 0 "#PWR071" H 3000 2050 50  0001 C CNN
 F 1 "GND" H 3000 2150 50  0000 C CNN
 F 2 "" H 3000 2300 50  0001 C CNN
@@
 	3000 2300 3000 1450
 $Comp
-L connectors:Rotated_Barrel J7
+L connectors:Rotated_Barrel J6
 U 1 1 5A779AD3
 P 3700 1500
-AR Path="/5A4C34AF/5A779AD3" Ref="J7"  Part="1"
-AR Path="/5A4C3F5F/5A779AD3" Ref="J8"  Part="1"
-F 0 "J8" H 3700 1710 50  0000 C CNN
+AR Path="/5A4C34AF/5A779AD3" Ref="J6"  Part="1"
+AR Path="/5A4C3F5F/5A779AD3" Ref="J7"  Part="1"
+F 0 "J7" H 3700 1710 50  0000 C CNN
 F 1 "Rotated_Barrel" H 3750 1350 50  0000 C CNN
 F 2 "Connectors:BARREL_JACK" H 3750 1440 50  0001 C CNN
@@
 Connection ~ 3450 1700
 $Comp
-L power:GND #PWR062
+L power:GND #PWR065
 U 1 1 5A77A9CB
 P 3450 2300
-AR Path="/5A4C34AF/5A77A9CB" Ref="#PWR062"  Part="1"
-AR Path="/5A4C3F5F/5A77A9CB" Ref="#PWR069"  Part="1"
-F 0 "#PWR069" H 3450 2050 50  0001 C CNN
+AR Path="/5A4C34AF/5A77A9CB" Ref="#PWR065"  Part="1"
+AR Path="/5A4C3F5F/5A77A9CB" Ref="#PWR072"  Part="1"
+F 0 "#PWR072" H 3450 2050 50  0001 C CNN
 F 1 "GND" H 3450 2150 50  0000 C CNN
 F 2 "" H 3450 2300 50  0001 C CNN
@@
 Connection ~ 1100 1050
 $Comp
-L power:GND #PWR057
+L power:GND #PWR060
 U 1 1 5A77D43C
 P 1100 2300
-AR Path="/5A4C34AF/5A77D43C" Ref="#PWR057"  Part="1"
-AR Path="/5A4C3F5F/5A77D43C" Ref="#PWR064"  Part="1"
-F 0 "#PWR064" H 1100 2050 50  0001 C CNN
+AR Path="/5A4C34AF/5A77D43C" Ref="#PWR060"  Part="1"
+AR Path="/5A4C3F5F/5A77D43C" Ref="#PWR067"  Part="1"
+F 0 "#PWR067" H 1100 2050 50  0001 C CNN
 F 1 "GND" H 1100 2150 50  0000 C CNN
 F 2 "" H 1100 2300 50  0001 C CNN
@@
 	4100 475  4100 2500
 $Comp
-L power:+48V #PWR056
+L power:+48V #PWR059
 U 1 1 5A84C99A
 P 1050 950
-AR Path="/5A4C34AF/5A84C99A" Ref="#PWR056"  Part="1"
-AR Path="/5A4C3F5F/5A84C99A" Ref="#PWR063"  Part="1"
-F 0 "#PWR063" H 1050 800 50  0001 C CNN
+AR Path="/5A4C34AF/5A84C99A" Ref="#PWR059"  Part="1"
+AR Path="/5A4C3F5F/5A84C99A" Ref="#PWR066"  Part="1"
+F 0 "#PWR066" H 1050 800 50  0001 C CNN
 F 1 "+48V" H 1050 1090 50  0000 C CNN
 F 2 "" H 1050 950 50  0001 C CNN
