File: Panel.sch (KiCad schematic (older format))
At the start: 10 parts, among them J6 Rotated_Barrel, U7 LM3406HV

Commit message: Made the Digikey more generic
Parts:
- C20, C21, C23: Buy (none) -> https://www.digikey.com/product-detail/en/samsung-electro-m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; Digikey https://www.digikey.com/product-detail/en/samsung-electro-m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 -> (none)
- C22: Buy (none) -> https://www.digikey.com/product-detail/en/kemet/C0805C223K5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; Digikey https://www.digikey.com/product-detail/en/kemet/C0805C223K5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 -> (none)
- D1: Buy (none) -> https://www.digikey.com/product-detail/en/nexperia-usa-inc/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; Digikey https://www.digikey.com/product-detail/en/nexperia-usa-inc/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 -> (none)
- L3: Buy (none) -> https://www.digikey.com/product-detail/en/taiyo-yuden/NS101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; Digikey https://www.digikey.com/product-detail/en/taiyo-yuden/NS101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 -> (none)
- R11: Buy (none) -> https://www.digikey.com/product-detail/en/yageo/RC0805FR-07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; Digikey https://www.digikey.com/product-detail/en/yageo/RC0805FR-07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 -> (none)
- R12: Buy (none) -> https://www.digikey.com/product-detail/en/panasonic-electro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; Digikey https://www.digikey.com/product-detail/en/panasonic-electro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 -> (none)
- U7: Buy (none) -> https://www.digikey.com/product-detail/en/texas-instruments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; Digikey https://www.digikey.com/product-detail/en/texas-instruments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 -> (none)
Changed lines of the file:
@@
 F 2 "Resistors_SMD:R_0603" V 1280 1300 50  0001 C CNN
 F 3 "" H 1350 1300 50  0001 C CNN
-F 4 "https://www.digikey.com/product-detail/en/yageo/RC0805FR-07162KL/311-162KCRCT-ND/730577" V 1350 1300 60  0001 C CNN "Digikey"
+F 4 "https://www.digikey.com/product-detail/en/yageo/RC0805FR-07162KL/311-162KCRCT-ND/730577" V 1350 1300 60  0001 C CNN "Buy"
 	1    1350 1300
 	1    0    0    -1
@@
 F 2 "Capacitors_SMD:C_0603" H 1500 2150 50  0001 C CNN
 F 3 "" H 1500 2150 50  0001 C CNN
-F 4 "https://www.digikey.com/product-detail/en/samsung-electro-mechanics/CL21B104KACNNNC/1276-1099-1-ND/3889185" H 1500 2150 60  0001 C CNN "Digikey"
+F 4 "https://www.digikey.com/product-detail/en/samsung-electro-mechanics/CL21B104KACNNNC/1276-1099-1-ND/3889185" H 1500 2150 60  0001 C CNN "Buy"
 	1    1500 2150
 	1    0    0    -1
@@
 F 2 "Capacitors_SMD:C_0603" H 2700 2150 50  0001 C CNN
 F 3 "" H 2700 2150 50  0001 C CNN
-F 4 "https://www.digikey.com/product-detail/en/samsung-electro-mechanics/CL21B104KACNNNC/1276-1099-1-ND/3889185" H 2700 2150 60  0001 C CNN "Digikey"
+F 4 "https://www.digikey.com/product-detail/en/samsung-electro-mechanics/CL21B104KACNNNC/1276-1099-1-ND/3889185" H 2700 2150 60  0001 C CNN "Buy"
 	1    2700 2150
 	1    0    0    -1
@@
 F 2 "Capacitors_SMD:C_0603" H 2450 850 50  0001 C CNN
 F 3 "" H 2450 850 50  0001 C CNN
-F 4 "https://www.digikey.com/product-detail/en/kemet/C0805C223K5RACTU/399-1163-1-ND/411438" H 2450 850 60  0001 C CNN "Digikey"
+F 4 "https://www.digikey.com/product-detail/en/kemet/C0805C223K5RACTU/399-1163-1-ND/411438" H 2450 850 60  0001 C CNN "Buy"
 	1    2450 850
 	0    -1   -1   0
@@
 F 2 "" H 3250 1050 50  0001 C CNN
 F 3 "" H 3250 1050 50  0001 C CNN
-F 4 "https://www.digikey.com/product-detail/en/taiyo-yuden/NS10145T330MNA/587-3126-1-ND/2774716" V 3250 1050 60  0001 C CNN "Digikey"
+F 4 "https://www.digikey.com/product-detail/en/taiyo-yuden/NS10145T330MNA/587-3126-1-ND/2774716" V 3250 1050 60  0001 C CNN "Buy"
 	1    3250 1050
 	0    -1   -1   0
@@
 F 2 "Diodes_SMD:D_SOD-123" H 3000 1300 50  0001 C CNN
 F 3 "" H 3000 1300 50  0001 C CNN
-F 4 "https://www.digikey.com/product-detail/en/nexperia-usa-inc/PMEG6020ER115/1727-5217-1-ND/2531816" H 3000 1300 60  0001 C CNN "Digikey"
+F 4 "https://www.digikey.com/product-detail/en/nexperia-usa-inc/PMEG6020ER115/1727-5217-1-ND/2531816" H 3000 1300 60  0001 C CNN "Buy"
 	1    3000 1300
 	0    1    1    0
@@
 F 2 "Resistors_SMD:R_0603" V 3380 1900 50  0001 C CNN
 F 3 "" H 3450 1900 50  0001 C CNN
-F 4 "https://www.digikey.com/product-detail/en/panasonic-electronic-components/ERJ-6DSFR16V/P19313CT-ND/6004668" V 3450 1900 60  0001 C CNN "Digikey"
+F 4 "https://www.digikey.com/product-detail/en/panasonic-electronic-components/ERJ-6DSFR16V/P19313CT-ND/6004668" V 3450 1900 60  0001 C CNN "Buy"
 	1    3450 1900
 	1    0    0    -1
@@
 F 2 "Capacitors_SMD:C_0603" H 1100 1300 50  0001 C CNN
 F 3 "" H 1100 1300 50  0001 C CNN
-F 4 "https://www.digikey.com/product-detail/en/samsung-electro-mechanics/CL31B105KCHNNNE/1276-1838-1-ND/3889924" H 1100 1300 60  0001 C CNN "Digikey"
+F 4 "https://www.digikey.com/product-detail/en/samsung-electro-mechanics/CL31B105KCHNNNE/1276-1838-1-ND/3889924" H 1100 1300 60  0001 C CNN "Buy"
 	1    1100 1300
 	1    0    0    -1
@@
 F 2 "Housings_SSOP:TSSOP-14_4.4x5mm_Pitch0.65mm" H 2100 2100 60  0001 C CNN
 F 3 "http://www.ti.com/lit/ds/symlink/lm3406.pdf" H 2100 2100 60  0001 C CNN
-F 4 "https://www.digikey.com/product-detail/en/texas-instruments/LM3406HVMHX-NOPB/LM3406HVMHX-NOPBCT-ND/3526958" H 2100 1500 60  0001 C CNN "Digikey"
+F 4 "https://www.digikey.com/product-detail/en/texas-instruments/LM3406HVMHX-NOPB/LM3406HVMHX-NOPBCT-ND/3526958" H 2100 1500 60  0001 C CNN "Buy"
 	1    2100 1500
 	1    0    0    -1
